File: XG_Mobile_Dock_Flow.kicad_sch (KiCad schematic)
At the start: 58 parts, among them J1 5-1775443-8, J13 39300240, J14 469911008, J17 8730, J2 20455-040E-76, J3 20455-040E-76, J4 3-2362375-4, J5 USB_C_Receptacle, SW1 SW_Push, U1 DS160PR410RNQR, U2 DS160PR410RNQR

Commit message: preparations for building, still need to sort out ac decoupling capacitators
Parts:
- J14: now in the parts list
Changed lines of the file:
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@@
 		(unit 1)
 		(exclude_from_sim no)
-		(in_bom no)
+		(in_bom yes)
 		(on_board yes)
 		(dnp no)

Commit message: final update, got some things wrongs, starting a new version in a new branch
Parts:
- removed C38, C39, C40, C41, C43, C44, C45, C46: 0.1μF, Capacitor_SMD:C_0402_1005Metric, symbol Device:C
- removed C42, C47: 1μF, Capacitor_SMD:C_0402_1005Metric, symbol Device:C
- added C17, C18, C19, C20, C22, C23, C24, C25: 0.1μF, Capacitor_SMD:C_0201_0603Metric, symbol Device:C
- added C21, C26: 1μF, Capacitor_SMD:C_0201_0603Metric, symbol Device:C
Connections:
- net +3V3: now also C17.2, C18.2, C19.2, C20.2, C21.2, C22.2, C23.2, C24.2, C25.2, C26.2
- net GND: now also C17.1, C18.1, C19.1, C20.1, C21.1, C22.1, C23.1, C24.1, C25.1, C26.1
