File: XG_Mobile_Dock_Redriver.kicad_pcb (KiCad board)
At the start: 4 copper layers, 220 x 65 mm, 153 parts, among them J1 5-1775443-8, J10 SWD, J11 UART, J12 I2C1, J13 39301240, J14 SWD, J15 SWD, J17 8730, J2 20455-040E-76, J20 SWD, J21 SWD, J22 SWD, J23 SWD, J24 SWD, J25 SWD, J26 SWD, J27 SWD, J28 SWD, J29 SWD, J3 20455-040E-76, J30 SWD, J31 SWD, J32 SWD, J33 SWD, J4 3-2362375-4, J5 USB_C_Receptacle, J6 455860005, Q16 AO3401A, Q17 2N7002W, SW1 SW_Push, U1 DS320PR810NJXR, U12 STM32F030C8Tx, U2 DS320PR810NJXR

Commit message: some fixes and added labels
Routing:
- net GND: vias 96 -> 100
Other:
- board text added: "CPU->GPU"
- board text added: "GPU->CPU"
- board text added: "L0"
- board text added: "L1"
- board text added: "L2"
- board text added: "L3"
