File: XG_Mobile_Dock_Redriver.kicad_pcb (KiCad board)
At the start: 4 copper layers, 220 x 65 mm, 151 parts, among them J1 5-1775443-8, J10 SWD, J11 UART, J12 I2C1, J13 39301240, J14 SWD, J15 SWD, J17 8730, J2 20455-040E-76, J20 SWD, J21 SWD, J22 SWD, J23 SWD, J24 SWD, J25 SWD, J26 SWD, J27 SWD, J28 SWD, J29 SWD, J3 20455-040E-76, J30 SWD, J31 SWD, J32 SWD, J33 SWD, J4 3-2362375-4, J5 USB_C_Receptacle, J6 455860005, Q16 AO3401A, Q17 2N7002W, SW1 SW_Push, U1 DS320PR810NJXR, U12 STM32F030C8Tx, U2 DS320PR810NJXR

Commit message: more tweaks
Parts:
- moved C33 1.14 mm to (102.2, 72.7)
- moved C39 0.97 mm to (106.4, 72.6)
- moved C41 0.69 mm to (115.5, 78.5), turned to 180 degrees
- moved C35 0.61 mm to (119.7, 78.6), turned to 0 degrees
- moved C40 0.18 mm to (106.4, 78.6)
- moved C36 0.16 mm to (119.7, 72.6)
- moved C38 0.12 mm to (115.5, 72.6)
- moved C34 0.12 mm to (102.2, 78.5)
Routing:
- net +3V3: track 273.2 -> 271.4 mm

Commit message: fixed pcb and more tweaks
Routing:
- net /HSO0P: track 2.49 -> 3.08 mm
- net /HSO0N: track 2.49 -> 3.08 mm
- net /HSO2P: track 2.45 -> 2.98 mm
- net /HSO2N: track 2.45 -> 2.98 mm
Changed lines of the file:
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@@
 	)
 	(via
-		(at 107.69 81.29)
+		(at 106.72 80.26)
 		(size 0.4)
 		(drill 0.3)
@@
 	)
 	(segment
-		(start 102.590203 64.723953)
-		(end 102.93666 64.377496)
+		(start 102.593543 65.052484)
+		(end 102.590203 65.049144)
 		(width 0.205486)
 		(layer "F.Cu")
@@
 	)
 	(segment
-		(start 102.93666 64.377496)
-		(end 102.93666 63.727496)
+		(start 102.91 65.904999)
+		(end 102.91 65.559998)
 		(width 0.205486)
 		(layer "F.Cu")
@@
 	)
 	(segment
-		(start 102.91 65.904999)
-		(end 102.91 65.559998)
+		(start 102.93666 64.253232)
+		(end 102.93666 63.727496)
 		(width 0.205486)
 		(layer "F.Cu")
@@
 	)
 	(segment
-		(start 102.590203 64.969144)
-		(end 102.590203 64.723953)
+		(start 102.93666 64.377496)
+		(end 102.93666 63.727496)
 		(width 0.205486)
 		(layer "F.Cu")
@@
 	)
 	(segment
-		(start 102.593543 64.972484)
-		(end 102.590203 64.969144)
+		(start 102.590203 64.723953)
+		(end 102.93666 64.377496)
 		(width 0.205486)
 		(layer "F.Cu")
@@
 	)
 	(segment
-		(start 102.91 65.559998)
-		(end 102.593543 65.243541)
+		(start 102.590203 65.049144)
+		(end 102.590203 64.723953)
 		(width 0.205486)
 		(layer "F.Cu")
@@
 	(segment
 		(start 102.593543 65.243541)
-		(end 102.593543 64.972484)
+		(end 102.593543 65.052484)
 		(width 0.205486)
 		(layer "F.Cu")
@@
 	)
 	(segment
-		(start 98.91 66)
-		(end 98.91 65.779263)
+		(start 102.91 65.559998)
+		(end 102.593543 65.243541)
 		(width 0.205486)
 		(layer "F.Cu")
-		(net 10)
+		(net 9)
 	)
 	(segment
-		(start 98.583543 65.2)
-		(end 98.590203 65.19334)
+		(start 98.91 65.654999)
+		(end 98.583543 65.328542)
 		(width 0.205486)
 		(layer "F.Cu")
@@
 	)
 	(segment
-		(start 98.678071 64.636085)
-		(end 98.93666 64.377496)
+		(start 98.583543 65.18)
+		(end 98.590203 65.17334)
 		(width 0.205486)
 		(layer "F.Cu")
@@
 	)
 	(segment
-		(start 98.590203 65.19334)
-		(end 98.590203 64.848217)
+		(start 98.590203 65.17334)
+		(end 98.590203 64.723953)
 		(width 0.205486)
 		(layer "F.Cu")
@@
 	)
 	(segment
-		(start 98.822132 65.567131)
-		(end 98.671411 65.41641)
+		(start 98.91 66)
+		(end 98.91 65.654999)
 		(width 0.205486)
 		(layer "F.Cu")
@@
 	)
 	(segment
-		(start 98.93666 64.377496)
-		(end 98.93666 63.727496)
+		(start 98.583543 65.328542)
+		(end 98.583543 65.18)
 		(width 0.205486)
 		(layer "F.Cu")
@@
 	)
 	(segment
-		(start 98.583543 65.204278)
-		(end 98.583543 65.2)
-		(width 0.205486)
-		(layer "F.Cu")
-		(net 10)
-	)
-	(arc
-		(start 98.583543 65.204278)
-		(mid 98.606379 65.319083)
-		(end 98.671411 65.41641)
-		(width 0.205486)
-		(layer "F.Cu")
-		(net 10)
-	)
-	(arc
-		(start 98.678071 64.636085)
-		(mid 98.613039 64.733412)
-		(end 98.590203 64.848217)
+		(start 98.590203 64.723953)
+		(end 98.93666 64.377496)
 		(width 0.205486)
 		(layer "F.Cu")
 		(net 10)
 	)
-	(arc
-		(start 98.822132 65.567131)
-		(mid 98.887164 65.664458)
-		(end 98.91 65.779263)
+	(segment
+		(start 98.93666 64.377496)
+		(end 98.93666 63.727496)
 		(width 0.205486)
 		(layer "F.Cu")
@@
 	)
 	(segment
-		(start 98.276457 65.082484)
-		(end 98.283117 65.075824)
+		(start 98.283117 64.723953)
+		(end 97.93666 64.377496)
 		(width 0.205486)
 		(layer "F.Cu")
@@
 	)
 	(segment
-		(start 98.276457 65.204278)
-		(end 98.276457 65.082484)
+		(start 97.93666 64.377496)
+		(end 97.93666 63.727496)
 		(width 0.205486)
 		(layer "F.Cu")
@@
 	(segment
 		(start 97.95 66)
-		(end 97.95 65.779263)
+		(end 97.95 65.654999)
 		(width 0.205486)
 		(layer "F.Cu")
@@
 	)
 	(segment
-		(start 98.195249 64.636085)
-		(end 97.93666 64.377496)
+		(start 98.283117 65.055824)
+		(end 98.283117 64.723953)
 		(width 0.205486)
 		(layer "F.Cu")
@@
 	)
 	(segment
-		(start 97.93666 64.377496)
-		(end 97.93666 63.727496)
+		(start 98.276457 65.328542)
+		(end 98.276457 65.062484)
 		(width 0.205486)
 		(layer "F.Cu")
@@
 	)
 	(segment
-		(start 98.037868 65.567131)
-		(end 98.188589 65.41641)
+		(start 97.95 65.654999)
+		(end 98.276457 65.328542)
 		(width 0.205486)
 		(layer "F.Cu")
@@
 	)
 	(segment
-		(start 98.283117 65.075824)
-		(end 98.283117 64.848217)
-		(width 0.205486)
-		(layer "F.Cu")
-		(net 19)
-	)
-	(arc
-		(start 97.95 65.779263)
-		(mid 97.972836 65.664458)
-		(end 98.037868 65.567131)
-		(width 0.205486)
-		(layer "F.Cu")
-		(net 19)
-	)
-	(arc
-		(start 98.276457 65.204278)
-		(mid 98.253621 65.319083)
-		(end 98.188589 65.41641)
-		(width 0.205486)
-		(layer "F.Cu")
-		(net 19)
-	)
-	(arc
-		(start 98.283117 64.848217)
-		(mid 98.260281 64.733412)
-		(end 98.195249 64.636085)
+		(start 98.276457 65.062484)
+		(end 98.283117 65.055824)
 		(width 0.205486)
 		(layer "F.Cu")
@@
 	)
 	(segment
-		(start 93.195249 64.636085)
-		(end 93.024528 64.465364)
-		(width 0.205486)
-		(layer "F.Cu")
-		(net 24)
-	)
-	(segment
 		(start 92.93666 64.253232)
 		(end 92.93666 63.727496)
@@
 	)
 	(segment
-		(start 93.283117 65.070824)
-		(end 93.283117 64.848217)
+		(start 93.283117 64.723953)
+		(end 92.93666 64.377496)
 		(width 0.205486)
 		(layer "F.Cu")
@@
 	)
 	(segment
-		(start 93.047868 65.567131)
-		(end 93.193589 65.42141)
+		(start 92.96 65.654999)
+		(end 93.281457 65.333542)
 		(width 0.205486)
 		(layer "F.Cu")
@@
 	)
 	(segment
-		(start 93.281457 65.209278)
-		(end 93.281457 65.072484)
+		(start 92.93666 64.377496)
+		(end 92.93666 63.727496)
 		(width 0.205486)
 		(layer "F.Cu")
@@
 	)
 	(segment
-		(start 92.96 66)
-		(end 92.96 65.779263)
+		(start 93.281457 65.102484)
+		(end 93.283117 65.100824)
 		(width 0.205486)
 		(layer "F.Cu")
@@
 	)
 	(segment
-		(start 93.281457 65.072484)
-		(end 93.283117 65.070824)
-		(width 0.205486)
-		(layer "F.Cu")
-		(net 24)
-	)
-	(arc
-		(start 93.283117 64.848217)
-		(mid 93.260281 64.733412)
-		(end 93.195249 64.636085)
+		(start 93.283117 65.100824)
+		(end 93.283117 64.723953)
 		(width 0.205486)
 		(layer "F.Cu")
 		(net 24)
 	)
-	(arc
-		(start 93.047868 65.567131)
-		(mid 92.982836 65.664458)
-		(end 92.96 65.779263)
-		(width 0.205486)
-		(layer "F.Cu")
-		(net 24)
-	)
-	(arc
-		(start 93.193589 65.42141)
-		(mid 93.258621 65.324083)
-		(end 93.281457 65.209278)
+	(segment
+		(start 92.96 66)
+		(end 92.96 65.654999)
 		(width 0.205486)
 		(layer "F.Cu")
 		(net 24)
 	)
-	(arc
-		(start 93.024528 64.465364)
-		(mid 92.959496 64.368037)
-		(end 92.93666 64.253232)
+	(segment
+		(start 93.281457 65.333542)
+		(end 93.281457 65.102484)
 		(width 0.205486)
 		(layer "F.Cu")
@@
 	)
 	(segment
-		(start 93.590203 65.18834)
-		(end 93.590203 64.848217)
-		(width 0.205486)
-		(layer "F.Cu")
-		(net 30)
-	)
-	(segment
-		(start 93.588543 65.209278)
-		(end 93.588543 65.19)
+		(start 93.590203 64.723953)
+		(end 93.93666 64.377496)
 		(width 0.205486)
 		(layer "F.Cu")
@@
 	)
 	(segment
-		(start 93.678071 64.636085)
-		(end 93.848792 64.465364)
+		(start 93.590203 65.21834)
+		(end 93.590203 64.723953)
 		(width 0.205486)
 		(layer "F.Cu")
@@
 	)
 	(segment
-		(start 93.822132 65.567131)
-		(end 93.676411 65.42141)
+		(start 93.93666 64.377496)
+		(end 93.93666 63.727496)
 		(width 0.205486)
 		(layer "F.Cu")
@@
 	)
 	(segment
-		(start 93.588543 65.19)
-		(end 93.590203 65.18834)
+		(start 93.91 65.654999)
+		(end 93.588543 65.333542)
 		(width 0.205486)
 		(layer "F.Cu")
@@
 	)
 	(segment
-		(start 93.91 66)
-		(end 93.91 65.779263)
+		(start 93.588543 65.22)
+		(end 93.590203 65.21834)
 		(width 0.205486)
 		(layer "F.Cu")
 		(net 30)
 	)
-	(arc
-		(start 93.93666 64.253232)
-		(mid 93.913824 64.368037)
-		(end 93.848792 64.465364)
-		(width 0.205486)
-		(layer "F.Cu")
-		(net 30)
-	)
-	(arc
-		(start 93.676411 65.42141)
-		(mid 93.611379 65.324083)
-		(end 93.588543 65.209278)
-		(width 0.205486)
-		(layer "F.Cu")
-		(net 30)
-	)
-	(arc
-		(start 93.678071 64.636085)
-		(mid 93.613039 64.733412)
-		(end 93.590203 64.848217)
+	(segment
+		(start 93.91 66)
+		(end 93.91 65.654999)
 		(width 0.205486)
 		(layer "F.Cu")
 		(net 30)
 	)
-	(arc
-		(start 93.822132 65.567131)
-		(mid 93.887164 65.664458)
-		(end 93.91 65.779263)
+	(segment
+		(start 93.588543 65.333542)
+		(end 93.588543 65.22)
 		(width 0.205486)
 		(layer "F.Cu")
@@
 	)
 	(segment
-		(start 102.286457 65.09)
-		(end 102.283117 65.08666)
+		(start 102.286457 65.17)
+		(end 102.283117 65.16666)
 		(width 0.205486)
 		(layer "F.Cu")
@@
 	)
 	(segment
-		(start 102.286457 65.243541)
-		(end 102.286457 65.09)
+		(start 101.97 65.559998)
+		(end 102.286457 65.243541)
 		(width 0.205486)
 		(layer "F.Cu")
@@
 	)
 	(segment
-		(start 101.97 65.559998)
-		(end 102.286457 65.243541)
+		(start 102.283117 65.16666)
+		(end 102.283117 64.723953)
 		(width 0.205486)
 		(layer "F.Cu")
@@
 	)
 	(segment
-		(start 102.283117 65.08666)
-		(end 102.283117 64.723953)
+		(start 102.286457 65.243541)
+		(end 102.286457 65.17)
 		(width 0.205486)
 		(layer "F.Cu")
@@
 	)
 	(segment
+		(start 101.93666 64.377496)
+		(end 101.93666 63.727496)
+		(width 0.205486)
+		(layer "F.Cu")
+		(net 31)
+	)
+	(segment
 		(start 101.93666 63.727496)
-		(end 101.93666 64.377496)
+		(end 101.93666 64.253232)
 		(width 0.205486)
 		(layer "F.Cu")
