File: XG_Mobile_Dock_XT.kicad_pcb (KiCad board)
At the start: 8 copper layers, 220.1 x 93 mm, 222 parts, among them IC1 PI2EQX22024XEAEX, J1 5-1775443-8, J10 SWD, J11 UART, J12 I2C1, J13 39301240, J14 I2C1, J2 20455-040E-76, J3 20455-040E-76, J5 USB_C_Receptacle, J6 455860005, J7 10147430-113T0LF, Q16 AO3401A, Q17 2N7002W, SW1 SW_Push, U1 DS320PR810NJXR, U12 STM32F030C8Tx, U2 DS320PR810NJXR

Commit message: tweaks
Routing:
- net GND: vias 2781 -> 2782
