File: XG_Mobile_Dock_Redriver_Single.kicad_pcb (KiCad board)
At the start: 6 copper layers, 220.1 x 93 mm, 156 parts, among them J1 5-1775443-8, J10 SWD, J11 UART, J12 I2C1, J13 39301240, J14 I2C1, J2 20455-040E-76, J3 20455-040E-76, J4 469911008, J7 10147430-113T0LF, Q16 AO3401A, Q17 2N7002W, SW1 SW_Push, U1 DS320PR810NJXR, U12 STM32F030C8Tx, U7 TPS7A8400ARGRR, U8 TPS7A8400ARGRR

Commit message: Update XG_Mobile_Dock_Redriver_Single.kicad_pcb
Parts:
- removed SW22, SW23: ~, DSWB03LHGET:SW-TH_DSWB03LHGET
Routing:
- net +3V3Redriver: track 131.4 -> 85.7 mm
- net Net-(U1-GAIN0/SDA): track 127.2 -> 144.7 mm
- net Net-(U1-RX_DET/SCL): track 140.0 -> 149.4 mm
- net Net-(U1-PD0): track 135.1 -> 138.5 mm
- net Net-(U1-PD1): track 146.8 -> 147.7 mm
