File: XG_Mobile_Dock_Dual_Redriver.kicad_pcb (KiCad board)
At the start: 6 copper layers, 220.1 x 93 mm, 207 parts, among them J1 5-1775443-8, J10 SWD, J11 UART, J12 I2C1, J13 39301240, J14 I2C1, J2 20455-040E-76, J3 20455-040E-76, J4 469911008, J7 10147430-113T0LF, Q16 AO3401A, Q17 2N7002W, SW1 SW_Push, U1 DS320PR810NJXR, U12 STM32F030C8Tx, U2 DS320PR810NJXR, U7 TPS7A8400ARGRR, U8 TPS7A8400ARGRR

Commit message: renamed boards
renamed boards
Other:
- board text added: "XG Mobile Dock Dual Redriver v0.8"
- board text removed: "XG Mobile Dock XT v0.8"
Changed lines of the file:
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@@
 		)
 	)
-	(gr_text "XG Mobile Dock XT v0.8"
+	(gr_text "XG Mobile Dock Dual Redriver v0.8"
 		(at 75.621496 55.121496 0)
 		(layer "F.SilkS")
