File: XG_Mobile_Dock_Single_Redriver.kicad_pcb (KiCad board)
At the start: 6 copper layers, 220.1 x 93 mm, 154 parts, among them J1 5-1775443-8, J10 SWD, J11 UART, J12 I2C1, J13 39301240, J14 I2C1, J2 20455-040E-76, J3 20455-040E-76, J4 469911008, J7 CEE016400140111, Q16 AO3401A, Q17 2N7002W, SW1 SW_Push, U1 DS320PR810NJXR, U12 STM32F030C8Tx, U7 TPS7A8400ARGRR, U8 TPS7A8400ARGRR

Commit message: better layout
Routing:
- net /C_DN: track 117.4 -> 114.6 mm
- net /C_DP: track 117.4 -> 114.6 mm
- net /C_RXP: track 130.1 -> 127.4 mm
- net /C_RXN: track 130.1 -> 127.5 mm
- net /C_TXP: track 110.1 -> 107.7 mm
- net /C_TXN: track 110.1 -> 107.7 mm
- net +3V3Redriver: track 85.7 -> 85.0 mm
- net /CPU_TO_GPU_EQ0_0: track 125.9 -> 125.4 mm
- net GND: vias 2536 -> 2533
