File: XG_Mobile_Dock_Retimer.kicad_pcb (KiCad board)
At the start: 6 copper layers, 220.1 x 93 mm, 118 parts, among them J1 5-1775443-8, J10 SWD, J11 UART, J12 I2C1, J13 39301240, J17 8730, J2 20455-040E-76, J3 20455-040E-76, J4 3-2362375-4, J5 USB_C_Receptacle, J6 455860005, Q16 AO3401A, Q17 2N7002W, SW1 SW_Push, U1 DS160PT801ACBR, U12 STM32F030C8Tx

Commit message: no message
Parts:
- moved C68 11.4 mm to (131.7, 98.5), turned to 90 degrees
- moved C69 11.4 mm to (132.4, 98.5), turned to 90 degrees
- moved C67 11.4 mm to (129.4, 98.5), turned to 90 degrees
- moved C66 11.4 mm to (128.7, 98.5), turned to 90 degrees
Routing:
- net /HSIT7N: track 0.00 -> 17.4 mm, vias 0 -> 1
- net /HSIT7P: track 0.00 -> 17.3 mm, vias 0 -> 1
- net /HSIT5N: track 0.00 -> 11.1 mm, vias 0 -> 1
- net /HSIT5P: track 0.00 -> 10.7 mm, vias 0 -> 1
- net /HSIT6N: track 5.99 -> 14.8 mm
- net /HSIT6P: track 6.47 -> 15.1 mm
- net /HSIL4P: track 77.0 -> 85.4 mm
- net /HSIL4N: track 77.7 -> 86.0 mm
- net /HSIL5P: track 83.9 -> 91.3 mm
- net /HSIL5N: track 84.6 -> 92.0 mm
- net /HSIL6P: track 91.6 -> 97.8 mm
- net /HSIL6N: track 92.3 -> 98.5 mm
- net /HSIL7P: track 85.4 -> 90.6 mm
- net /HSIL7N: track 85.9 -> 91.2 mm
- net /HSI6P: track 0.00 -> 3.52 mm, vias 0 -> 1
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
Commit message: Update XG_Mobile_Dock_Retimer.kicad_pcb
Routing:
- net GND: vias 163 -> 185

Commit message: Update XG_Mobile_Dock_Retimer.kicad_pcb
Routing:
- net GND: vias 185 -> 200
