File: MCU_Retimer.kicad_sch (KiCad schematic)
At the start: 31 parts, among them J10 SWD, J11 UART, J12 I2C1, Q16 AO3401A, Q17 2N7002W, U12 STM32F030C8Tx

Commit message: eeeeeeeee
eeeeeeeee
Parts:
- added C31, C32, C33, C34: 0.1µF, Capacitor_SMD:C_0402_1005Metric, symbol Device:C
- added U4: ~, STM32F103RCT6:LQFP-64_L10.0-W10.0-P0.50-LS12.0-BL, symbol STM32F103RCT6:STM32F103RCT6
Connections:
- net +3V3MCU: now also C31.2, C32.2, C33.2, C34.2, U4.13 (VDDA), U4.32 (VDD_1), U4.48 (VDD_2), U4.64 (VDD_3); no longer U12.1 (VDD), U12.24 (VDD), U12.48 (VDD), U12.9 (VDDA)
- net FAN_ON: now also U4.45 (PA12); no longer U12.33 (PA12)
- net GND: now also C31.1, C32.1, C33.1, C34.1, U4.12 (VSSA), U4.18 (VSS_4), U4.31 (VSS_1), U4.47 (VSS_2), U4.63 (VSS_3)
- net PA0: now also U4.14 (PA0-WKUP); no longer U12.10 (PA0)
- net PA1: now also U4.15 (PA1); no longer U12.11 (PA1)
- net PA15: now also U4.50 (PA15); no longer U12.38 (PA15)
- net PA2: now also U4.16 (PA2); no longer U12.12 (PA2)
- net PA3: now also U4.17 (PA3); no longer U12.13 (PA3)
- net PA4: now also U4.20 (PA4); no longer U12.14 (PA4)
- net PA5: now also U4.21 (PA5); no longer U12.15 (PA5)
- net PA7: now also U4.23 (PA7); no longer U12.17 (PA7)
- net PC13: now also U4.2 (PC13-TAMPER-RTC); no longer U12.2 (PC13)
- net PC14: now also U4.3 (PC14-OSC32_IN); no longer U12.3 (PC14)
- net PC15: now also U4.4 (PC15-OSC32_OUT); no longer U12.4 (PC15)
- net RX: now also U4.43 (PA10); no longer U12.31 (PA10)
- net SWCLK: now also U4.49 (PA14); no longer U12.37 (PA14)
- net SWDIO: now also U4.46 (PA13); no longer U12.34 (PA13)
- net TX: now also U4.42 (PA9); no longer U12.30 (PA9)
- net ~{RST}: now also U4.7 (NRST); no longer U12.7 (NRST)
- net at U12.44 (BOOT0): no longer R84.2
- new net: R84.2, U4.60 (BOOT0)
Other:
- moved on the sheet: J10, J11, R84, R85

Commit message: Update MCU_Retimer.kicad_sch
Parts:
- removed C112, C113, C114: 0.1µF, Capacitor_SMD:C_0402_1005Metric, symbol Device:C
- removed C115: 10nF, Capacitor_SMD:C_0402_1005Metric, symbol Device:C
- removed C117: 4.7µF, Capacitor_SMD:C_0402_1005Metric, symbol Device:C
- removed C118: 1µF, Capacitor_SMD:C_0402_1005Metric, symbol Device:C
- removed U12: STM32F030C8Tx, Package_QFP:LQFP-48_7x7mm_P0.5mm, symbol MCU_ST_STM32F0:STM32F030C8Tx
- added C35: 10nF, Capacitor_SMD:C_0402_1005Metric, symbol Device:C
- added C36: 1µF, Capacitor_SMD:C_0402_1005Metric, symbol Device:C
- added C74: 4.7µF, Capacitor_SMD:C_0402_1005Metric, symbol Device:C
Connections:
- net GND is gone; now on net +3V3MCU: C128.2, C129.2, C130.2, C31.1, C32.1, C33.1, C34.1, D15.2 (A), J10.4 (Pin_4), J11.4 (Pin_4), J12.4 (Pin_4), J18.1 (Pin_1), J19.1 (Pin_1), Q17.2 (S), R84.1, TH1.2, U4.12 (VSSA), U4.18 (VSS_4), U4.31 (VSS_1), U4.47 (VSS_2), U4.63 (VSS_3)
- net +3V3MCU: now also C35.1, C35.2, C36.1, C36.2, C74.1, C74.2
- net FAN_ON: now also U4.41 (PA8); no longer U4.45 (PA12)
- net FAN_PWM: now also U4.55 (PB3)
- net PB12: now also U4.33 (PB12)
- net PB13: now also U4.34 (PB13)
- net PB14: now also U4.35 (PB14)
- net PB15: now also U4.36 (PB15)
- net PB2: now also U4.28 (PB2)
- net PB4: now also U4.56 (PB4)
- net PB5: now also U4.57 (PB5)
- net PB6: now also U4.58 (PB6)
- net PF0: now also U4.37 (PC6)
- net PF1: now also U4.38 (PC7)
- net SCL1: now also U4.61 (PB8)
- net SCL2: now also U4.29 (PB10)
- net SDA1: now also U4.62 (PB9)
- net SDA2: now also U4.30 (PB11)
- net ~{CASE_LED}: now also U4.39 (PC8)
- net at R86.1, TH1.1: now also U4.27 (PB1)
- net USBDM: now reaches U4.44 (PA11)
- new net USBDP: U4.45 (PA12)
Other:
- moved on the sheet: C32, C33, C34, J10, J11, J12, J16, R19, R20, R33, R34, R74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

Commit message: eeeeeeee
eeeeeeee
Parts:
- added C75, C76: 15pF, Capacitor_SMD:C_0402_1005Metric, symbol Device:C
- added CRYSTAL1: 8MHz, CF4008M00012001:CRYSTAL-SMD_4P-L3.2-W2.5-BL_SIT8008BI, symbol CF4008M00012001:CF4008M00012001
- added R16: 250, Resistor_SMD:R_0402_1005Metric, symbol Device:R_Small
Connections:
- net +3V3MCU: now also C75.1, C76.2, CRYSTAL1.2 (GND), CRYSTAL1.4 (GND)
- net at U4.5 (PD0-OSC_IN): now also C75.2, CRYSTAL1.3
- net at U4.6 (PD1-OSC_OUT): now also R16.2
- new net: C76.1, CRYSTAL1.1, R16.1
Other:
- moved on the sheet: R85

Commit message: fixes
fixes
Connections:
- net +3V3MCU: no longer C128.2, C129.2, C130.2, C31.1, C32.1, C33.1, C34.1, C35.1, C36.1, C74.1, C75.1, C76.2, CRYSTAL1.2 (GND), CRYSTAL1.4 (GND), D15.2 (A), J10.4 (Pin_4), J11.4 (Pin_4), J12.4 (Pin_4), J18.1 (Pin_1), J19.1 (Pin_1), Q17.2 (S), R84.1, TH1.2, U4.12 (VSSA), U4.18 (VSS_4), U4.31 (VSS_1), U4.47 (VSS_2), U4.63 (VSS_3)
- new net GND: C128.2, C129.2, C130.2, C31.1, C32.1, C33.1, C34.1, C35.1, C36.1, C74.1, C75.1, C76.2, CRYSTAL1.2 (GND), CRYSTAL1.4 (GND), D15.2 (A), J10.4 (Pin_4), J11.4 (Pin_4), J12.4 (Pin_4), J18.1 (Pin_1), J19.1 (Pin_1), Q17.2 (S), R84.1, TH1.2, U4.12 (VSSA), U4.18 (VSS_4), U4.31 (VSS_1), U4.47 (VSS_2), U4.63 (VSS_3)
Changed lines of the file:
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@@
 	)
 	(junction
-		(at 27.94 53.34)
-		(diameter 0)
-		(color 0 0 0 0)
-	)
-	(junction
 		(at 201.93 63.5)
 		(diameter 0)
@@
 	(wire
 		(pts
-			(xy 25.4 53.34) (xy 27.94 53.34)
-		)
-		(stroke
-			(width 0)
-			(type default)
-		)
-	)
-	(wire
-		(pts
 			(xy 68.58 53.34) (xy 68.58 58.42)
 		)
@@
 					(unit 1)
 				)
-			)
-		)
-	)
-	(symbol
-		(lib_id "power:GND")
-		(at 25.4 53.34 270)
-		(unit 1)
-		(exclude_from_sim no)
-		(in_bom yes)
-		(on_board yes)
-		(dnp no)
-		(fields_autoplaced yes)
-		(property "Reference" "#PWR063"
-			(at 19.05 53.34 0)
-			(effects
-				(font
-					(size 1.27 1.27)
-				)
-				(hide yes)
-			)
-		)
-		(property "Value" "GND"
-			(at 21.59 53.3399 90)
-			(effects
-				(font
-					(size 1.27 1.27)
-				)
-				(justify right)
-			)
-		)
-		(property "Footprint" ""
-			(at 25.4 53.34 0)
-			(effects
-				(font
-					(size 1.27 1.27)
-				)
-				(hide yes)
-			)
-		)
-		(property "Datasheet" ""
-			(at 25.4 53.34 0)
-			(effects
-				(font
-					(size 1.27 1.27)
-				)
-				(hide yes)
-			)
-		)
-		(property "Description" "Power symbol creates a global label with name \"GND\" , ground"
-			(at 25.4 53.34 0)
-			(effects
-				(font
-					(size 1.27 1.27)
-				)
-				(hide yes)
-			)
-		)
-		(pin "1"
-		)
-		(instances
-			(project "MCU_Retimer"
-				(path "/e44dba81-61f4-41e9-92bb-329e30057892"
-					(reference "#PWR?")
-					(unit 1)
-				)
-			)
-			(project "XG_Mobile_Dock_Retimer"
-				(path "/f97e6956-ab08-42cb-8fed-03fa58e87f0e/ee7d8714-c34c-4773-b74b-c8779559fec9"
-					(reference "#PWR063")
-					(unit 1)
-				)

Commit message: eeee
Parts:
- added C86: 0.1µF, Capacitor_SMD:C_0402_1005Metric, symbol Device:C
- added L4, L5: FBMJ2125HS420-T, FBMJ2125HS420-T:L0805, symbol FBMJ2125HS420-T:FBMJ2125HS420-T
Connections:
- net +3V3MCU: now also U4.19 (VDD_4), C86.2, L4.1; no longer C34.2, U4.13 (VDDA)
- net GND: now also C86.1, L5.1; no longer U4.12 (VSSA)
- new net: L5.2, U4.12 (VSSA)
- new net: C34.2, L4.2, U4.13 (VDDA)

Commit message: eeeeeeeee
eeeeeeeee
Parts:
- removed C33, C86: 0.1µF, Capacitor_SMD:C_0402_1005Metric, symbol Device:C
- removed C35: 10nF, Capacitor_SMD:C_0402_1005Metric, symbol Device:C
- removed C36: 1µF, Capacitor_SMD:C_0402_1005Metric, symbol Device:C
- removed C74: 4.7µF, Capacitor_SMD:C_0402_1005Metric, symbol Device:C
- removed L4, L5: FBMJ2125HS420-T, FBMJ2125HS420-T:L0805, symbol FBMJ2125HS420-T:FBMJ2125HS420-T
- removed U4: ~, STM32F103RCT6:LQFP-64_L10.0-W10.0-P0.50-LS12.0-BL, symbol STM32F103RCT6:STM32F103RCT6
- added 1, 11: ~, STM32F405RGT6:LQFP-64_L10.0-W10.0-P0.50-LS12.0-BL, symbol STM32F405RGT6:STM32F405RGT6
- added C100, C101: 2.2µF, Capacitor_SMD:C_0603_1608Metric, symbol Device:C
- added C94, C95, C96, C97, C98: 0.1µF, Capacitor_SMD:C_0402_1005Metric, symbol Device:C
- added C99: 4.7µF, Capacitor_SMD:C_0402_1005Metric, symbol Device:C
- C31: value 0.1µF -> 1µF; LCSC C307331 -> C1592; Part_Number CL05B104KB54PNC -> CL10A105KO8NNNC
Connections:
- net +3V3MCU: now also C31.1, 11.1 (VBAT), 11.13 (VDDA), 11.19 (VDD), 11.32 (VDD), 11.48 (VDD), 11.64 (VDD), C94.2, C95.2, C96.2, C97.2, C98.2, C99.1; no longer C31.2
- net FAN_ON: now also 1.41 (PA8)
- net FAN_PWM: now also 1.55 (PB3(JTDOTRACESWO))
- net GND: now also C31.2, C34.2, 11.12 (VSSA), 11.18 (VSS), 11.63 (VSS), C100.1, C101.1, C94.1, C95.1, C96.1, C97.1, C98.1, C99.2; no longer C31.1, C34.1
- net PA0: now also 1.14 (PA0-WKUP(PA0))
- net PA1: now also 1.15 (PA1)
- net PA15: now also 1.50 (PA15(JTDI))
- net PA2: now also 1.16 (PA2)
- net PA3: now also 1.17 (PA3)
- net PA4: now also 1.20 (PA4)
- net PA5: now also 1.21 (PA5)
- net PA7: now also 1.23 (PA7)
- net PB12: now also 1.33 (PB12)
- net PB13: now also 1.34 (PB13)
- net PB14: now also 1.35 (PB14)
- net PB15: now also 1.36 (PB15)
- net PB2: now also 1.28 (PB2-BOOT1(PB2))
- net PB4: now also 1.56 (PB4(NJTRST))
- net PB5: now also 1.57 (PB5)
- net PB6: now also 1.58 (PB6)
- net PC13: now also 1.2 (PC13)
- net PC14: now also 1.3 (PC14-OSC32_IN(PC14))
- net PC15: now also 1.4 (PC15-OSC32_OUT(PC15))
- net PF0: now also 1.37 (PC6)
- net PF1: now also 1.38 (PC7)
- net RX: now also 1.43 (PA10)
- net SCL1: now also 1.61 (PB8)
- net SCL2: now also 1.29 (PB10)
- net SDA1: now also 1.62 (PB9)
- net SDA2: now also 1.30 (PB11)
- net SWCLK: now also 1.49 (PA14(JTCK-SWCLK))
- net SWDIO: now also 1.46 (PA13(JTMS-SWDIO))
- net TX: now also 1.42 (PA9)
- net USBDM: now also 1.44 (PA11)
- net USBDP: now also 1.45 (PA12)
- net ~{CASE_LED}: now also 1.39 (PC8)
- net ~{RST}: now also C34.1, 1.7 (NRST)
- net at C75.2, CRYSTAL1.3: now also 1.5 (PH0-OSC_IN(PH0))
- net at R16.2: now also 1.6 (PH1-OSC_OUT(PH1))
- net at R86.1, TH1.1: now also 1.27 (PB1)
- net at R84.2: now also 1.60 (BOOT0)
- new net: 1.47 (VCAP_2), C100.2
- new net: 1.31 (VCAP_1), C101.2
Other:
- moved on the sheet: C75, C76, CRYSTAL1, J10, J11, J12, R16, R84, R85, R86, TH1

Commit message: eeeeee
eeeeeee
Parts:
- renumbered 1 to U12, 11 to U12
Changed lines of the file:
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@@
 		(dnp no)
 		(fields_autoplaced yes)
-		(property "Reference" "1"
+		(property "Reference" "U12"
 			(at 73.66 20.32 0)
 			(effects
@@
 			(project ""
 				(path "/f97e6956-ab08-42cb-8fed-03fa58e87f0e/ee7d8714-c34c-4773-b74b-c8779559fec9"
-					(reference "1")
+					(reference "U12")
 					(unit 1)
 				)
@@
 		(dnp no)
 		(fields_autoplaced yes)
-		(property "Reference" "11"
+		(property "Reference" "U12"
 			(at 74.93 127 0)
 			(effects
@@
 			(project ""
 				(path "/f97e6956-ab08-42cb-8fed-03fa58e87f0e/ee7d8714-c34c-4773-b74b-c8779559fec9"
-					(reference "11")
+					(reference "U12")
 					(unit 2)
 				)
