File: MCU_Retimer.kicad_sch (KiCad schematic)
At the start: 40 parts, among them J10 SWD, J11 UART, J12 I2C1, Q16 AO3401A, Q17 2N7002W

Commit message: no message
Connections:
- net PC2: now reaches U12.10 (PC2)
- net PC3: now reaches U12.11 (PC3)
- net PC0: now reaches U12.8 (PC0)
- net PC1: now reaches U12.9 (PC1)
Changed lines of the file:
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@@
+		)
+	)
+	(hierarchical_label "PC2"
+		(shape bidirectional)
+		(at 50.8 78.74 180)
+		(effects
+			(font
+				(size 1.27 1.27)
+			)
+			(justify right)
 		)
 	)
@@
 		(shape bidirectional)
 		(at 50.8 60.96 180)
+		(effects
+			(font
+				(size 1.27 1.27)
+			)
+			(justify right)
+		)
+	)
+	(hierarchical_label "PC3"
+		(shape bidirectional)
+		(at 50.8 81.28 180)
 		(effects
 			(font
@@
 			)
 			(justify left)
+		)
+	)
+	(hierarchical_label "PC0"
+		(shape bidirectional)
+		(at 50.8 73.66 180)
+		(effects
+			(font
+				(size 1.27 1.27)
+			)
+			(justify right)
 		)
 	)
@@
 		)
 	)
+	(hierarchical_label "PC1"
+		(shape bidirectional)
+		(at 50.8 76.2 180)
+		(effects
+			(font
+				(size 1.27 1.27)
+			)
+			(justify right)
+		)
+	)

Commit message: eeeeeeeee
eeeeeeeeee
Connections:
- net PC11: now reaches U12.52 (PC11)
- net PC12: now reaches U12.53 (PC12)
Changed lines of the file:
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@@
+		)
+	)
+	(hierarchical_label "PC11"
+		(shape bidirectional)
+		(at 50.8 104.14 180)
+		(effects
+			(font
+				(size 1.27 1.27)
+			)
+			(justify right)
 		)
 	)
@@
 		(effects
 			(font
+				(size 1.27 1.27)
+			)
+			(justify right)
+		)
+	)
+	(hierarchical_label "PC12"
+		(shape bidirectional)
+		(at 50.8 106.68 180)
+		(effects
+			(font

Commit message: eee
eee
Parts:
- R16: value 250 -> 150; LCSC C2909342 -> C25082; Part_Number FRC0402F2700TS -> 0402WGF1500TCE
Changed lines of the file:
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@@
 			)
 		)
-		(property "Value" "250"
+		(property "Value" "150"
 			(at 110.4901 81.28 0)
 			(effects
@@
 			)
 		)
-		(property "Part_Number" "FRC0402F2700TS"
+		(property "Part_Number" "0402WGF1500TCE"
 			(at 111.76 83.82 0)
 			(effects
@@
 			)
 		)
-		(property "LCSC" "C2909342"
+		(property "LCSC" "C25082"
 			(at 111.76 83.82 0)
 			(effects

Commit message: eeee
eeee
Connections:
- net PC11 is gone; now on net RX: U12.52 (PC11)
- net RX: no longer U12.43 (PA10)
- net TX: now also U12.51 (PC10); no longer U12.42 (PA9)
- new net USBVBUS: U12.42 (PA9)
Other:
- moved on the sheet: J11
Changed lines of the file:
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@@
 	(wire
 		(pts
-			(xy 24.13 50.8) (xy 24.13 49.53)
+			(xy 24.13 99.06) (xy 24.13 97.79)
 		)
 		(stroke
@@
 	(wire
 		(pts
-			(xy 24.13 58.42) (xy 22.86 58.42)
+			(xy 24.13 106.68) (xy 22.86 106.68)
 		)
 		(stroke
@@
 	(wire
 		(pts
-			(xy 22.86 50.8) (xy 24.13 50.8)
+			(xy 22.86 99.06) (xy 24.13 99.06)
 		)
 		(stroke
@@
 	(wire
 		(pts
-			(xy 24.13 59.69) (xy 24.13 58.42)
+			(xy 24.13 107.95) (xy 24.13 106.68)
 		)
 		(stroke
@@
 	(wire
 		(pts
-			(xy 22.86 55.88) (xy 50.8 55.88)
+			(xy 22.86 104.14) (xy 50.8 104.14)
 		)
 		(stroke
@@
 	(wire
 		(pts
-			(xy 50.8 53.34) (xy 22.86 53.34)
+			(xy 50.8 101.6) (xy 22.86 101.6)
 		)
 		(stroke
@@
 	)
 	(label "TX"
-		(at 49.53 53.34 180)
+		(at 49.53 101.6 180)
 		(effects
 			(font
@@
 	)
 	(label "RX"
-		(at 49.53 55.88 180)
+		(at 49.53 104.14 180)
 		(effects
 			(font
@@
 		)
 	)
-	(hierarchical_label "PC11"
-		(shape bidirectional)
-		(at 50.8 104.14 180)
-		(effects
-			(font
-				(size 1.27 1.27)
-			)
-			(justify right)
-		)
-	)
 	(hierarchical_label "PA7"
 		(shape bidirectional)
@@
 		)
 	)
+	(hierarchical_label "USBVBUS"
+		(shape bidirectional)
+		(at 50.8 53.34 180)
+		(effects
+			(font
+				(size 1.27 1.27)
+			)
+			(justify right)
+		)
+	)
 	(hierarchical_label "PA15"
 		(shape bidirectional)
@@
 	(symbol
 		(lib_id "power:+3V3")
-		(at 24.13 49.53 0)
+		(at 24.13 97.79 0)
 		(mirror y)
 		(unit 1)
@@
 		(dnp no)
 		(property "Reference" "#PWR01"
-			(at 24.13 53.34 0)
+			(at 24.13 101.6 0)
 			(effects
 				(font
@@
 		)
 		(property "Value" "+3V3MCU"
-			(at 24.13 45.212 0)
+			(at 24.13 93.472 0)
 			(effects
 				(font
@@
 		)
 		(property "Footprint" ""
-			(at 24.13 49.53 0)
+			(at 24.13 97.79 0)
 			(effects
 				(font
@@
 		)
 		(property "Datasheet" ""
-			(at 24.13 49.53 0)
+			(at 24.13 97.79 0)
 			(effects
 				(font
@@
 		)
 		(property "Description" "Power symbol creates a global label with name \"+3V3\""
-			(at 24.13 49.53 0)
+			(at 24.13 97.79 0)
 			(effects
 				(font
@@
 	(symbol
 		(lib_id "power:GND")
-		(at 24.13 59.69 0)
+		(at 24.13 107.95 0)
 		(mirror y)
 		(unit 1)
@@
 		(dnp no)
 		(property "Reference" "#PWR036"
-			(at 24.13 66.04 0)
+			(at 24.13 114.3 0)
 			(effects
 				(font
@@
 		)
 		(property "Value" "GND"
-			(at 21.844 63.5 0)
+			(at 21.844 111.76 0)
 			(effects
 				(font
@@
 		)
 		(property "Footprint" ""
-			(at 24.13 59.69 0)
+			(at 24.13 107.95 0)
 			(effects
 				(font
@@
 		)
 		(property "Datasheet" ""
-			(at 24.13 59.69 0)
+			(at 24.13 107.95 0)
 			(effects
 				(font
@@
 		)
 		(property "Description" "Power symbol creates a global label with name \"GND\" , ground"
-			(at 24.13 59.69 0)
+			(at 24.13 107.95 0)
 			(effects
 				(font
@@
 	(symbol
 		(lib_id "Connector_Generic:Conn_01x04")
-		(at 17.78 53.34 0)
+		(at 17.78 101.6 0)
 		(mirror y)
 		(unit 1)
@@
 		(fields_autoplaced yes)
 		(property "Reference" "J11"
-			(at 15.24 53.3399 0)
+			(at 15.24 101.5999 0)
 			(effects
 				(font
@@
 		)
 		(property "Value" "UART"
-			(at 15.24 55.8799 0)
+			(at 15.24 104.1399 0)
 			(effects
 				(font
@@
 		)
 		(property "Footprint" "Connector_PinHeader_2.54mm:PinHeader_1x04_P2.54mm_Vertical"
-			(at 17.78 53.34 0)
+			(at 17.78 101.6 0)
 			(effects
 				(font
@@
 		)
 		(property "Datasheet" "~"
-			(at 17.78 53.34 0)
+			(at 17.78 101.6 0)
 			(effects
 				(font
@@
 		)
 		(property "Description" "Generic connector, single row, 01x04, script generated (kicad-library-utils/schlib/autogen/connector/)"
-			(at 17.78 53.34 0)
+			(at 17.78 101.6 0)
 			(effects
 				(font
@@
 		)
 		(property "Part_Number" "2.54-1*4"
-			(at 17.78 53.34 0)
+			(at 17.78 101.6 0)
 			(effects
 				(font
@@
 		)
 		(property "LCSC" "C5116483"
-			(at 17.78 53.34 0)
+			(at 17.78 101.6 0)
 			(effects
 				(font
@@
 		)
 		(property "Sim.Device" ""
-			(at 17.78 53.34 0)
+			(at 17.78 101.6 0)
 			(effects
 				(font
@@
 		)
 		(property "Sim.Pins" ""
-			(at 17.78 53.34 0)
+			(at 17.78 101.6 0)
 			(effects
 				(font
@@
 		)
 		(property "Sim.Type" ""
-			(at 17.78 53.34 0)
+			(at 17.78 101.6 0)
 			(effects
 				(font

Commit message: eeeeeeeeee
eeeeeeee
Connections:
- net PA6: now reaches U12.22 (PA6)
- net PC4: now reaches U12.24 (PC4)
- net PC5: now reaches U12.25 (PC5)
- net PB0: now reaches U12.26 (PB0)
- net PC9: now reaches U12.40 (PC9)
- net PD2: now reaches U12.54 (PD2)
- net PB7: now reaches U12.59 (PB7)
Changed lines of the file:
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@@
+		)
+	)
+	(hierarchical_label "PC5"
+		(shape bidirectional)
+		(at 50.8 86.36 180)
+		(effects
+			(font
+				(size 1.27 1.27)
+			)
+			(justify right)
 		)
 	)
@@
 		)
 	)
+	(hierarchical_label "PB7"
+		(shape bidirectional)
+		(at 96.52 45.72 0)
+		(effects
+			(font
+				(size 1.27 1.27)
+			)
+			(justify left)
+		)
+	)
 	(hierarchical_label "PA0"
 		(shape bidirectional)
@@
 		)
 	)
+	(hierarchical_label "PC4"
+		(shape bidirectional)
+		(at 50.8 83.82 180)
+		(effects
+			(font
+				(size 1.27 1.27)
+			)
+			(justify right)
+		)
+	)
+	(hierarchical_label "PB0"
+		(shape bidirectional)
+		(at 96.52 27.94 0)
+		(effects
+			(font
+				(size 1.27 1.27)
+			)
+			(justify left)
+		)
+	)
 	(hierarchical_label "USBVBUS"
 		(shape bidirectional)
@@
 		(shape bidirectional)
 		(at 50.8 73.66 180)
+		(effects
+			(font
+				(size 1.27 1.27)
+			)
+			(justify right)
+		)
+	)
+	(hierarchical_label "PA6"
+		(shape bidirectional)
+		(at 50.8 43.18 180)
 		(effects
 			(font
@@
 		)
 	)
+	(hierarchical_label "PD2"
+		(shape bidirectional)
+		(at 96.52 73.66 0)
+		(effects
+			(font
+				(size 1.27 1.27)
+			)
+			(justify left)
+		)
+	)
 	(hierarchical_label "PF1"
 		(shape bidirectional)
@@
 		)
 	)
+	(hierarchical_label "PC9"
+		(shape bidirectional)
+		(at 50.8 99.06 180)
+		(effects
+			(font
+				(size 1.27 1.27)
+			)
+			(justify right)
+		)
+	)

Commit message: eeee
eeeee
Parts:
- added R46: 1k, Resistor_SMD:R_0402_1005Metric, symbol Device:R_Small
- added SW3: ~, DSWB02LHGET:SW-TH_DSWB02LHGET, symbol DSWB02LHGET:DSWB02LHGET
Connections:
- net +3V3MCU: now also R46.1
- net at R84.2: now also SW3.3; no longer U12.60 (BOOT0)
- new net: R46.2, SW3.4
- new net BOOT0: SW3.1, SW3.2, U12.60 (BOOT0)
Other:
- moved on the sheet: R84
