File: XG_Mobile_Dock_Retimer.kicad_sch (KiCad schematic)
At the start: 248 parts, among them J1 5-1775443-8, J13 39301240, J14 469911008, J17 8730, J2 20455-040E-76, J3 20455-040E-76, J7 CEE016400140111, SW1 SW_Push, U1 DS160PT801ACBR, U2 TPS7A8400ARGRR, U7 TPS7A8400ARGRR

Commit message: eee
eee
Parts:
- added C203, C207: 10uF, Capacitor_SMD:C_0402_1005Metric, symbol Device:C
- added C204, C205, C206: 100nF, Capacitor_SMD:C_0201_0603Metric, symbol Device:C
- C92: footprint Capacitor_SMD:C_0805_2012Metric -> Capacitor_SMD:C_0402_1005Metric; LCSC C15850 -> C15525; Part_Number CL21A106KAYNNNE -> CL05A106MQ5NUNC
Connections:
- net +1V17_2: now also C92.2, C203.2, C204.2, C205.2, C206.2, C207.2; no longer C92.1
- net GND: now also C92.1, C203.1, C204.1, C205.1, C206.1, C207.1; no longer C92.2

Commit message: eee
eee
Parts:
- removed J17: 8730, KEYSTONE_8730:KEYSTONE_8730, symbol KEYSTONE_8730:8730
- added U4, U6: ~, CONN-SMD_T31000:CONN-SMD_T31000, symbol T31000:T31000
Connections:
- net GND: now also U4.1, U6.1
Changed lines of the file:
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@@
 	(wire
 		(pts
-			(xy 287.02 29.21) (xy 287.02 34.29)
-		)
-		(stroke
-			(width 0)
-			(type default)
-		)
-	)
-	(wire
-		(pts
 			(xy 218.44 215.9) (xy 218.44 218.44)
 		)
@@
 	)
 	(symbol
-		(lib_id "KEYSTONE_8730:8730")
-		(at 297.18 29.21 0)
+		(lib_id "T31000:T31000")
+		(at 45.72 298.45 0)
 		(unit 1)
 		(exclude_from_sim no)
@@
 		(dnp no)
 		(fields_autoplaced yes)
-		(property "Reference" "J17"
-			(at 303.53 27.9399 0)
+		(property "Reference" "U4"
+			(at 49.53 297.8149 0)
 			(effects
 				(font
@@
 			)
 		)
-		(property "Value" "8730"
-			(at 303.53 30.4799 0)
+		(property "Value" "~"
+			(at 49.53 299.72 0)
 			(effects
 				(font
@@
 			)
 		)
-		(property "Footprint" "KEYSTONE_8730:KEYSTONE_8730"
-			(at 297.18 29.21 0)
+		(property "Footprint" "CONN-SMD_T31000:CONN-SMD_T31000"
+			(at 45.72 298.45 0)
 			(effects
 				(font
 					(size 1.27 1.27)
 				)
-				(justify bottom)
 				(hide yes)
 			)
 		)
-		(property "Datasheet" ""
-			(at 297.18 29.21 0)
+		(property "Datasheet" "https://atta.szlcsc.com/upload/public/pdf/source/20200107/C481468_C71AD29EE3547CB6EB2C94611C55257F.pdf"
+			(at 45.72 298.45 0)
 			(effects
 				(font
@@
 		)
 		(property "Description" ""
-			(at 297.18 29.21 0)
-			(effects
-				(font
-					(size 1.27 1.27)
-				)
-				(hide yes)
-			)
-		)
-		(property "PARTREV" "C"
-			(at 297.18 29.21 0)
-			(effects
-				(font
-					(size 1.27 1.27)
-				)
-				(justify bottom)
-				(hide yes)
-			)
-		)
-		(property "SNAPEDA_PN" "8730"
-			(at 297.18 29.21 0)
-			(effects
-				(font
-					(size 1.27 1.27)
-				)
-				(justify bottom)
-				(hide yes)
-			)
-		)
-		(property "STANDARD" "Manufacturer Recommendations"
-			(at 297.18 29.21 0)
-			(effects
-				(font
-					(size 1.27 1.27)
-				)
-				(justify bottom)
-				(hide yes)
-			)
-		)
-		(property "MAXIMUM_PACKAGE_HEIGHT" "6.25 mm"
-			(at 297.18 29.21 0)
+			(at 45.72 298.45 0)
 			(effects
 				(font
 					(size 1.27 1.27)
 				)
-				(justify bottom)
 				(hide yes)
 			)
 		)
-		(property "MANUFACTURER" "Keystone"
-			(at 297.18 29.21 0)
+		(property "Manufacturer" "XFCN(兴飞)"
+			(at 45.72 298.45 0)
 			(effects
 				(font
 					(size 1.27 1.27)
 				)
-				(justify bottom)
 				(hide yes)
 			)
 		)
-		(property "Sim.Device" ""
-			(at 297.18 29.21 0)
+		(property "Part_Number" "T31000"
+			(at 45.72 298.45 0)
 			(effects
 				(font
@@
 			)
 		)
-		(property "Sim.Pins" ""
-			(at 297.18 29.21 0)
-			(effects
-				(font
-					(size 1.27 1.27)
-				)
-				(hide yes)
-			)
-		)
-		(property "Sim.Type" ""
-			(at 297.18 29.21 0)
+		(property "LCSC" "C481468"
+			(at 45.72 298.45 0)
 			(effects
 				(font
@@
 		)
 		(instances
-			(project "XG_Mobile_Dock_Lite"
+			(project "XG_Mobile_Dock_Retimer"
 				(path "/f97e6956-ab08-42cb-8fed-03fa58e87f0e"
-					(reference "J17")
+					(reference "U4")
 					(unit 1)
 				)
@@
 	)
 	(symbol
+		(lib_id "power:GND")
+		(at 40.64 313.69 270)
+		(unit 1)
+		(exclude_from_sim no)
+		(in_bom yes)
+		(on_board yes)
+		(dnp no)
+		(fields_autoplaced yes)
+		(property "Reference" "#PWR071"
+			(at 34.29 313.69 0)
+			(effects
+				(font
+					(size 1.27 1.27)
+				)
+				(hide yes)
+			)
+		)
+		(property "Value" "GND"
+			(at 36.83 313.6899 90)
+			(effects
+				(font
+					(size 1.27 1.27)
+				)
+				(justify right)
+			)
+		)
+		(property "Footprint" ""
+			(at 40.64 313.69 0)
+			(effects
+				(font
+					(size 1.27 1.27)
+				)
+				(hide yes)
+			)
+		)
+		(property "Datasheet" ""
+			(at 40.64 313.69 0)
+			(effects
+				(font
+					(size 1.27 1.27)
+				)
+				(hide yes)
+			)
+		)
+		(property "Description" "Power symbol creates a global label with name \"GND\" , ground"
+			(at 40.64 313.69 0)
+			(effects
+				(font
+					(size 1.27 1.27)
+				)
+				(hide yes)
+			)
+		)
+		(pin "1"
+		)
+		(instances
+			(project "XG_Mobile_Dock_Retimer"
+				(path "/f97e6956-ab08-42cb-8fed-03fa58e87f0e"
+					(reference "#PWR071")
+					(unit 1)
+				)
+			)
+		)
+	)
+	(symbol
 		(lib_id "Device:C")
 		(at 524.51 332.74 0)
@@
 	(symbol
 		(lib_id "power:GND")
+		(at 40.64 298.45 270)
+		(unit 1)
+		(exclude_from_sim no)
+		(in_bom yes)
+		(on_board yes)
+		(dnp no)
+		(fields_autoplaced yes)
+		(property "Reference" "#PWR070"
+			(at 34.29 298.45 0)
+			(effects
+				(font
+					(size 1.27 1.27)
+				)
+				(hide yes)
+			)
+		)
+		(property "Value" "GND"
+			(at 36.83 298.4499 90)
+			(effects
+				(font
+					(size 1.27 1.27)
+				)
+				(justify right)
+			)
+		)
+		(property "Footprint" ""
+			(at 40.64 298.45 0)
+			(effects
+				(font
+					(size 1.27 1.27)
+				)
+				(hide yes)
+			)
+		)
+		(property "Datasheet" ""
+			(at 40.64 298.45 0)
+			(effects
+				(font
+					(size 1.27 1.27)
+				)
+				(hide yes)
+			)
+		)
+		(property "Description" "Power symbol creates a global label with name \"GND\" , ground"
+			(at 40.64 298.45 0)
+			(effects
+				(font
+					(size 1.27 1.27)
+				)
+				(hide yes)
+			)
+		)
+		(pin "1"
+		)
+		(instances
+			(project "XG_Mobile_Dock_Retimer"
+				(path "/f97e6956-ab08-42cb-8fed-03fa58e87f0e"
+					(reference "#PWR070")
+					(unit 1)
+				)
+			)
+		)
+	)
+	(symbol
+		(lib_id "power:GND")
 		(at 82.55 140.97 90)
 		(unit 1)
@@
 	)
 	(symbol
+		(lib_id "T31000:T31000")
+		(at 45.72 313.69 0)
+		(unit 1)
+		(exclude_from_sim no)
+		(in_bom yes)
+		(on_board yes)
+		(dnp no)
+		(fields_autoplaced yes)
+		(property "Reference" "U6"
+			(at 49.53 313.0549 0)
+			(effects
+				(font
+					(size 1.27 1.27)
+				)
+				(justify left)
+			)
+		)
+		(property "Value" "~"
+			(at 49.53 314.96 0)
+			(effects
+				(font
+					(size 1.27 1.27)
+				)
+				(justify left)
+			)
+		)
+		(property "Footprint" "CONN-SMD_T31000:CONN-SMD_T31000"
+			(at 45.72 313.69 0)
+			(effects
+				(font
+					(size 1.27 1.27)
+				)
+				(hide yes)
+			)
+		)
+		(property "Datasheet" "https://atta.szlcsc.com/upload/public/pdf/source/20200107/C481468_C71AD29EE3547CB6EB2C94611C55257F.pdf"
+			(at 45.72 313.69 0)
+			(effects
+				(font
+					(size 1.27 1.27)
+				)
+				(hide yes)
+			)
+		)
+		(property "Description" ""
+			(at 45.72 313.69 0)
+			(effects
+				(font
+					(size 1.27 1.27)
+				)
+				(hide yes)
+			)
+		)
+		(property "Manufacturer" "XFCN(兴飞)"
+			(at 45.72 313.69 0)
+			(effects
+				(font
+					(size 1.27 1.27)
+				)
+				(hide yes)
+			)
+		)
+		(property "Part_Number" "T31000"
+			(at 45.72 313.69 0)
+			(effects
+				(font
+					(size 1.27 1.27)
+				)
+				(hide yes)
+			)
+		)
+		(property "LCSC" "C481468"
+			(at 45.72 313.69 0)
+			(effects
+				(font
+					(size 1.27 1.27)
+				)
+				(hide yes)
+			)
+		)
+		(pin "1"
+		)
+		(instances
+			(project "XG_Mobile_Dock_Retimer"
+				(path "/f97e6956-ab08-42cb-8fed-03fa58e87f0e"
+					(reference "U6")
+					(unit 1)
+				)
+			)
+		)
+	)
+	(symbol
 		(lib_id "power:GND")
 		(at 342.9 278.13 270)
@@
 					(unit 1)
 				)
-			)
-		)
-	)
-	(symbol
-		(lib_id "power:GND")
-		(at 287.02 34.29 0)
-		(unit 1)
-		(exclude_from_sim no)
-		(in_bom yes)
-		(on_board yes)
-		(dnp no)
-		(fields_autoplaced yes)
-		(property "Reference" "#PWR0100"
-			(at 287.02 40.64 0)
-			(effects
-				(font
-					(size 1.27 1.27)
-				)
-				(hide yes)
-			)
-		)
-		(property "Value" "GND"
-			(at 287.02 39.37 0)
-			(effects
-				(font
-					(size 1.27 1.27)
-				)
-			)
-		)
-		(property "Footprint" ""
-			(at 287.02 34.29 0)
-			(effects
-				(font
-					(size 1.27 1.27)
-				)
-				(hide yes)
-			)
-		)
-		(property "Datasheet" ""
-			(at 287.02 34.29 0)
-			(effects
-				(font
-					(size 1.27 1.27)
-				)
-				(hide yes)
-			)
-		)
-		(property "Description" "Power symbol creates a global label with name \"GND\" , ground"
-			(at 287.02 34.29 0)
-			(effects
-				(font
-					(size 1.27 1.27)
-				)
-				(hide yes)
-			)
-		)
-		(pin "1"
-		)
-		(instances
-			(project "XG_Mobile_Dock_Lite"
-				(path "/f97e6956-ab08-42cb-8fed-03fa58e87f0e"
-					(reference "#PWR0100")
-					(unit 1)
-				)

Commit message: EEEE
EEEEE
Parts:
- added SW2: ~, SS-12D10L5:SW-TH_SS-12D10L5, symbol SS-12D10L5:SS-12D10L5
Connections:
- net +3V3: now also SW2.3
- net BUCK_ON: now also SW2.2
- new net BUCK_ON_MCU: SW2.1
Changed lines of the file:
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@@
 		)
 	)
+	(label "BUCK_ON"
+		(at 332.74 300.99 0)
+		(effects
+			(font
+				(size 1.27 1.27)
+			)
+			(justify left bottom)
+		)
+	)
 	(label "HSOL0N"
 		(at 193.04 392.43 180)
@@
 		)
 	)
+	(label "BUCK_ON_MCU"
+		(at 137.16 8.89 180)
+		(effects
+			(font
+				(size 1.27 1.27)
+			)
+			(justify right bottom)
+		)
+	)
 	(label "LOCK_SW"
 		(at 40.64 29.21 0)
@@
 		)
 	)
+	(label "BUCK_ON_MCU"
+		(at 332.74 295.91 0)
+		(effects
+			(font
+				(size 1.27 1.27)
+			)
+			(justify left bottom)
+		)
+	)
 	(label "HSI0N"
 		(at 158.75 369.57 0)
@@
 		)
 	)
+	(global_label "+3V3"
+		(shape output)
+		(at 332.74 306.07 0)
+		(fields_autoplaced yes)
+		(effects
+			(font
+				(size 1.27 1.27)
+			)
+			(justify left)
+		)
+		(property "Intersheetrefs" "${INTERSHEET_REFS}"
+			(at 340.8052 306.07 0)
+			(effects
+				(font
+					(size 1.27 1.27)
+				)
+				(justify left)
+				(hide yes)
+			)
+		)
+	)
 	(global_label "+12V"
 		(shape input)
@@
 					(unit 1)
 				)
+			)
+		)
+	)
+	(symbol
+		(lib_id "SS-12D10L5:SS-12D10L5")
+		(at 330.2 300.99 270)
+		(unit 1)
+		(exclude_from_sim no)
+		(in_bom yes)
+		(on_board yes)
+		(dnp no)
+		(fields_autoplaced yes)
+		(property "Reference" "SW2"
+			(at 329.1206 308.61 0)
+			(effects
+				(font
+					(size 1.27 1.27)
+				)
+				(justify left)
+			)
+		)
+		(property "Value" "~"
+			(at 327.2155 308.61 0)
+			(effects
+				(font
+					(size 1.27 1.27)
+				)
+				(justify left)
+			)
+		)
+		(property "Footprint" "SS-12D10L5:SW-TH_SS-12D10L5"
+			(at 330.2 300.99 0)
+			(effects
+				(font
+					(size 1.27 1.27)
+				)
+				(hide yes)
+			)
+		)
+		(property "Datasheet" "https://item.szlcsc.com/datasheet/SS-12D10L5/300104.html"
+			(at 330.2 300.99 0)
+			(effects
+				(font
+					(size 1.27 1.27)
+				)
+				(hide yes)
+			)
+		)
+		(property "Description" "Circuit:SPDT Actuator Style:Rectangular Columnar Termination Style:PC Pin Length:13mm Width:6.8mm Switch Height:6.4mm Mounting Type:Through Hole Actuator Color:Black Current Rating:3A Voltage Rating:125V Life:10,000 Cycles Operating Temperature:-40°C~+85°C"
+			(at 330.2 300.99 0)
+			(effects
+				(font
+					(size 1.27 1.27)
+				)
+				(hide yes)
+			)
+		)
+		(property "Part_Number" "SS-12D10L5"
+			(at 330.2 300.99 0)
+			(effects
+				(font
+					(size 1.27 1.27)
+				)
+				(hide yes)
+			)
+		)
+		(property "Manufacturer" "XKB Connection(中国星坤)"
+			(at 330.2 300.99 0)
+			(effects
+				(font
+					(size 1.27 1.27)
+				)
+				(hide yes)
+			)
+		)
+		(property "LCSC" "C319012"
+			(at 330.2 300.99 0)
+			(effects
+				(font
+					(size 1.27 1.27)
+				)
+				(hide yes)
+			)
+		)
+		(pin "3"
+		)
+		(pin "1"
+		)
+		(pin "2"
+		)
+		(instances
+			(project "XG_Mobile_Dock_Retimer"
+				(path "/f97e6956-ab08-42cb-8fed-03fa58e87f0e"
+					(reference "SW2")
+					(unit 1)
+				)

Commit message: eeee
eeee
Parts:
- added C208: 0.1μF, Capacitor_SMD:C_0402_1005Metric, symbol Device:C
- added D1: H5VU25U, AZ1045-04F:AZ1045-04F, symbol AZ1045-04F:AZ1045-04F
- added R35, R36: 5.1k, Resistor_SMD:R_0402_1005Metric, symbol Device:R
- added U8: ~, GT-USB-7091A:USB-C-SMD_GT-USB-7091A, symbol GT-USB-7091A:GT-USB-7091A
Connections:
- net GND: now also C208.2, D1.3 (GND), D1.8 (GND), R35.1, R36.1, U8.1 (EH), U8.2 (EH), U8.3 (EH), U8.4 (EH), U8.A1 (GND), U8.A12 (GND), U8.B1 (GND), U8.B12 (GND)
- new net: R36.2, U8.B5 (CC2)
- new net: R35.2, U8.A5 (CC1)
- new net USBDN: D1.4 (I/O_3), D1.7 (NC), U8.A7 (D-)
- new net USBDP: D1.5 (I/O_4), D1.6 (NC), U8.A6 (D+)
- new net VBUS_USB2: C208.1, U8.A4 (VBUS), U8.A9 (VBUS), U8.B4 (VBUS), U8.B9 (VBUS)
- no-connect marks 21 -> 25

Commit message: eeee
eeee
Parts:
- added R37: 42.2k, Resistor_SMD:R_0402_1005Metric, symbol Device:R
- added R38: 100k, Resistor_SMD:R_0603_1608Metric, symbol Device:R
Connections:
- net GND: now also R38.1
- net VBUS_USB2: now also R37.2
- new net USBVBUS: R37.1, R38.2
Other:
- sheet MCU_Retimer ports: added USBVBUS; removed PC11

Commit message: eeeeee
eeeee
Parts:
- added R39: 42.2k, Resistor_SMD:R_0402_1005Metric, symbol Device:R
Connections:
- net +3V3MCU: now also R39.2
- net PGOOD_BUCK: now reaches U3.35 (PGOOD)
- net PGOOD_BUCK: now also R39.1

Commit message: eeeee
eeeee
Connections:
- net VBUS_USB2: now also D1.2 (I/O_2), D1.9 (NC)
- no-connect marks 25 -> 23
Changed lines of the file:
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@@
 	)
 	(no_connect
-		(at 215.9 -43.18)
-	)
-	(no_connect
 		(at 544.83 34.29)
 	)
@@
 	)
 	(no_connect
-		(at 243.84 -43.18)
-	)
-	(no_connect
 		(at 514.35 148.59)
 	)
@@
 	(wire
 		(pts
+			(xy 215.9 -43.18) (xy 243.84 -43.18)
+		)
+		(stroke
+			(width 0)
+			(type default)
+		)
+	)
+	(wire
+		(pts
 			(xy 264.16 336.55) (xy 275.59 336.55)
 		)
@@
 		(effects
 			(font
+				(size 1.27 1.27)
+			)
+			(justify left bottom)
+		)
+	)
+	(label "VBUS_USB2"
+		(at 243.84 -43.18 0)
+		(effects
+			(font

Commit message: eeeeeeee
eeeee
Parts:
- C24: footprint Capacitor_SMD:C_1206_3216Metric -> Capacitor_SMD:C_0603_1608Metric; LCSC C3908730 -> C51412; Part_Number CL31B335KOHNNNE -> CL10A335KP8NNNC
- C26: footprint Capacitor_SMD:C_1206_3216Metric -> Capacitor_SMD:C_0402_1005Metric; LCSC C2167327 -> C88946; Part_Number C1206C474K4RACTU -> GRM155R71A474KE01D
Changed lines of the file:
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@@
 	(generator_version "9.0")
 	(paper "A2")
-	(text "10nF 0201B103K250NT MfPArt C285010 LCSC 0201\n100nF GRM033R61C104KE84D MfPart C76937 LCSC 0201\n220nF GRM033R61C224KE14D MfPart C161474 LCSC 0201\n1uf CL03A105MO3NRNH MfPart C307385 LCSC LCSC 0201\n1k 1206W4F1001T5E MfPart C4410 LCSC 1206 Footprint\n430 0603WAF4300T5E MfPart C23170 LCSC 0603 Footprint\n30 0603WAF300JT5E MfPart C22985 LCSC 0603 Footprint\n3 0603WAF300KT5E MfPart C23157 LCSC 0603 Footprint\n240 0603WAF2400T5E MfPart C23350 LCSC 0603 Footprint\n10 0603WAF100JT5E MfPart C22859 LCSC 0603 Footprint\n4.7 uF CL10A475KP8NNNC MfPart C1705 LCSC 0603 Footprint\n60O @ 100Mhz BLM41PG600SN1L MfPArt C85844 LCSC 1806 Footprint\n100k 0.1% RT0603BRD07100KL MfPart C122538 LCSC 0603 Footprint\n133k 0.1% RT0402BRD07133KL MfPart C852517 LCSC 0402 Footprint\n22.1k 0.1% RT0603BRD0722K1L MfPart C723484 LCSC 0603 Footprint\n174 0.1%  ARG02BTC1740 MfPart C5266100 LCSC 0402 Footprint\n10k 0.1% RT0402BRD0710KL MfPart C190095 LCSC 0402 Footprint\n22uF TMK316BBJ226ML-T MfPart C386093 LCSC 1206 Footprint\n4.7uF GRM188C81E475KE11D MfPArt C417145 LCSC 0603 Footprint\n1uF GRM155R61E105KA12D MfPart C77009 LCSC 0402 Footprint\n0.1uF 50V CL05B104KB54PNC MfPart C307331 LCSC 0402 Footprint\n200uF 6.3V GRM31CR60J227ME11L MfPart C412252 LCSC 1206 Footprint\n100uF 6.3V CL31A107MQHNNNE MfPart C15008 LCSC 1206 Footprint\n47uF 6.3V C3216X7S0J476MT000E MfPart C342599 LCSC 1206 Footprint\n10uF 10V CL21A106KPFNNNE MfPArt C17024 LCSC 0805 Footprint\n3.3uF 16V CL31B335KOHNNNE MfPart C3908730 LCSC 1206 Footprint\n1uf 25V GRM155R61E105KA12D MfPart C77009 LCSC 0402 Footprint\n0.47uF 16V C1206C474K4RACTU MfPart C2167327 LCSC 1206 Footprint\n0.1uF 25V GRM155R71E104KE14D MfPart C77014 LCSC 0402 Footprint\n42.2k RT0402BRD0742K2L MfPart C852782 LCSC 0402 Footprint\n30.1k RT0402BRD0730K1L MfPart C852714 LCSC 0402 Footprint\n1 0805W8J010JT5E MfPart C25288 LCSC 0805 Footprint\n1nF CC0402JRX7R9BB102 Mfpart C93920 LCSC 0402 Footprint\n1 1% CRCW04021R00FKEDC MfPart C2077765 LCSC 0402 Footprint\n33 1% RC-01W33R0FT MfPart C320843 LCSC 0201 Footprint\n10uF CL05A106MQ5NUNC MfPart C15525 LCSC 0402 Footprint\n5.k 0603WAF5101T5E MfPart C23186 LCSC 0603 Footprint"
+	(text "10nF 0201B103K250NT MfPArt C285010 LCSC 0201\n100nF GRM033R61C104KE84D MfPart C76937 LCSC 0201\n220nF GRM033R61C224KE14D MfPart C161474 LCSC 0201\n1uf CL03A105MO3NRNH MfPart C307385 LCSC LCSC 0201\n1k 1206W4F1001T5E MfPart C4410 LCSC 1206 Footprint\n430 0603WAF4300T5E MfPart C23170 LCSC 0603 Footprint\n30 0603WAF300JT5E MfPart C22985 LCSC 0603 Footprint\n3 0603WAF300KT5E MfPart C23157 LCSC 0603 Footprint\n240 0603WAF2400T5E MfPart C23350 LCSC 0603 Footprint\n10 0603WAF100JT5E MfPart C22859 LCSC 0603 Footprint\n4.7 uF CL10A475KP8NNNC MfPart C1705 LCSC 0603 Footprint\n60O @ 100Mhz BLM41PG600SN1L MfPArt C85844 LCSC 1806 Footprint\n100k 0.1% RT0603BRD07100KL MfPart C122538 LCSC 0603 Footprint\n133k 0.1% RT0402BRD07133KL MfPart C852517 LCSC 0402 Footprint\n22.1k 0.1% RT0603BRD0722K1L MfPart C723484 LCSC 0603 Footprint\n174 0.1%  ARG02BTC1740 MfPart C5266100 LCSC 0402 Footprint\n10k 0.1% RT0402BRD0710KL MfPart C190095 LCSC 0402 Footprint\n22uF TMK316BBJ226ML-T MfPart C386093 LCSC 1206 Footprint\n4.7uF GRM188C81E475KE11D MfPArt C417145 LCSC 0603 Footprint\n1uF GRM155R61E105KA12D MfPart C77009 LCSC 0402 Footprint\n0.1uF 50V CL05B104KB54PNC MfPart C307331 LCSC 0402 Footprint\n200uF 6.3V GRM31CR60J227ME11L MfPart C412252 LCSC 1206 Footprint\n100uF 6.3V CL31A107MQHNNNE MfPart C15008 LCSC 1206 Footprint\n47uF 6.3V C3216X7S0J476MT000E MfPart C342599 LCSC 1206 Footprint\n10uF 10V CL21A106KPFNNNE MfPArt C17024 LCSC 0805 Footprint\n3.3uF 16V CL10A335KP8NNNC MfPart C51412 LCSC 0603 Footprint\n1uf 25V GRM155R61E105KA12D MfPart C77009 LCSC 0402 Footprint\n0.47uF 16V GRM155R71A474KE01D MfPart C88946 LCSC 0402 Footprint\n0.1uF 25V GRM155R71E104KE14D MfPart C77014 LCSC 0402 Footprint\n42.2k RT0402BRD0742K2L MfPart C852782 LCSC 0402 Footprint\n30.1k RT0402BRD0730K1L MfPart C852714 LCSC 0402 Footprint\n1 0805W8J010JT5E MfPart C25288 LCSC 0805 Footprint\n1nF CC0402JRX7R9BB102 Mfpart C93920 LCSC 0402 Footprint\n1 1% CRCW04021R00FKEDC MfPart C2077765 LCSC 0402 Footprint\n33 1% RC-01W33R0FT MfPart C320843 LCSC 0201 Footprint\n10uF CL05A106MQ5NUNC MfPart C15525 LCSC 0402 Footprint\n5.k 0603WAF5101T5E MfPart C23186 LCSC 0603 Footprint"
 		(exclude_from_sim no)
 		(at 420.624 20.574 0)
@@
 			)
 		)
-		(property "Footprint" "Capacitor_SMD:C_1206_3216Metric"
+		(property "Footprint" "Capacitor_SMD:C_0402_1005Metric"
 			(at 411.1752 298.45 0)
 			(effects
@@
 			)
 		)
-		(property "Part_Number" "C1206C474K4RACTU"
+		(property "Part_Number" "GRM155R71A474KE01D"
 			(at 410.21 302.26 0)
 			(effects
@@
 			)
 		)
-		(property "LCSC" "C2167327"
+		(property "LCSC" "C88946"
 			(at 410.21 302.26 0)
 			(effects
@@
 			)
 		)
-		(property "Footprint" "Capacitor_SMD:C_1206_3216Metric"
+		(property "Footprint" "Capacitor_SMD:C_0603_1608Metric"
 			(at 416.2552 298.45 0)
 			(effects
@@
 					(size 1.27 1.27)
 				)
-				(hide yes)
 			)
 		)
@@
 			)
 		)
-		(property "Part_Number" "CL31B335KOHNNNE"
+		(property "Part_Number" "CL10A335KP8NNNC"
 			(at 415.29 302.26 0)
 			(effects
@@
 			)
 		)
-		(property "LCSC" "C3908730"
+		(property "LCSC" "C51412"
 			(at 415.29 302.26 0)
 			(effects
