File: XG_Mobile_Dock_Quad_Redriver.kicad_sch (KiCad schematic)
At the start: 202 parts, among them J1 5-1775443-8, J13 39301240, J14 I2C1, J2 20455-040E-76, J3 20455-040E-76, J5 353180820, J7 CEE016400140111, SW1 SW_Push, U1 DS160PR410RNQR, U2 DS160PR410RNQR, U6 DS160PR410RNQR, U7 TPS7A8400ARGRR, U8 TPS7A8400ARGRR, U9 DS160PR410RNQR

Commit message: eeeeeee
eeee
Parts:
- U1, U2, U6, U9: value DS160PR410RNQR -> DS160PR410RNQT; LCSC (none) -> C2873337; Part_Number (none) -> DS160PR410RNQT
Changed lines of the file:
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@@
 			)
 		)
-		(property "Value" "DS160PR410RNQR"
+		(property "Value" "DS160PR410RNQT"
 			(at 161.29 318.77 0)
 			(effects
@@
 			)
 		)
-		(property "Datasheet" "DS160PR410RNQR"
+		(property "Datasheet" "DS160PR410RNQT"
 			(at 128.27 326.39 0)
 			(effects
@@
 			)
 		)
+		(property "Part_Number" "DS160PR410RNQT"
+			(at 128.27 326.39 0)
+			(effects
+				(font
+					(size 1.27 1.27)
+				)
+				(hide yes)
+			)
+		)
+		(property "LCSC" "C2873337"
+			(at 128.27 326.39 0)
+			(effects
+				(font
+					(size 1.27 1.27)
+				)
+				(hide yes)
+			)
+		)
 		(pin "18"
 		)
@@
 			)
 		)
-		(property "Value" "DS160PR410RNQR"
+		(property "Value" "DS160PR410RNQT"
 			(at 161.29 391.16 0)
 			(effects
@@
 			)
 		)
-		(property "Datasheet" "DS160PR410RNQR"
+		(property "Datasheet" "DS160PR410RNQT"
 			(at 128.27 398.78 0)
 			(effects
@@
 			)
 		)
+		(property "Part_Number" "DS160PR410RNQT"
+			(at 128.27 398.78 0)
+			(effects
+				(font
+					(size 1.27 1.27)
+				)
+				(hide yes)
+			)
+		)
+		(property "LCSC" "C2873337"
+			(at 128.27 398.78 0)
+			(effects
+				(font
+					(size 1.27 1.27)
+				)
+				(hide yes)
+			)
+		)
 		(pin "18"
 		)
@@
 			)
 		)
-		(property "Value" "DS160PR410RNQR"
+		(property "Value" "DS160PR410RNQT"
 			(at 525.78 430.53 0)
 			(effects
@@
 			)
 		)
-		(property "Datasheet" "DS160PR410RNQR"
+		(property "Datasheet" "DS160PR410RNQT"
 			(at 492.76 438.15 0)
 			(effects
@@
 			)
 		)
+		(property "Part_Number" "DS160PR410RNQT"
+			(at 492.76 438.15 0)
+			(effects
+				(font
+					(size 1.27 1.27)
+				)
+				(hide yes)
+			)
+		)
+		(property "LCSC" "C2873337"
+			(at 492.76 438.15 0)
+			(effects
+				(font
+					(size 1.27 1.27)
+				)
+				(hide yes)
+			)
+		)
 		(pin "18"
 		)
@@
 			)
 		)
-		(property "Value" "DS160PR410RNQR"
+		(property "Value" "DS160PR410RNQT"
 			(at 538.48 335.28 0)
 			(effects
@@
 			)
 		)
-		(property "Datasheet" "DS160PR410RNQR"
+		(property "Datasheet" "DS160PR410RNQT"
 			(at 505.46 342.9 0)
 			(effects
@@
 			(at 505.46 342.9 0)
 			(effects
+				(font
+					(size 1.27 1.27)
+				)
+				(hide yes)
+			)
+		)
+		(property "Part_Number" "DS160PR410RNQT"
+			(at 505.46 342.9 0)
+			(effects
+				(font
+					(size 1.27 1.27)
+				)
+				(hide yes)
+			)
+		)
+		(property "LCSC" "C2873337"
+			(at 505.46 342.9 0)
+			(effects

Commit message: eee
eeee
Parts:
- added C101, C102, C103, C104, C105, C106, C107, C108: 1uF, Capacitor_SMD:C_0201_0603Metric, symbol Device:C
- LED1, Q1, Q2, Q3, SW10, SW11, SW12, SW13, SW14, SW17, SW18, SW19, SW2, SW20, SW21, SW22, SW23, SW26, SW27, SW28, SW3, SW30, SW4, SW5, SW6, SW7, SW8, SW9, U3, U4, U5: value ~ -> (none)
Connections:
- net +3V3Redriver: now also C101.2, C102.2, C103.2, C104.2, C105.2, C106.2, C107.2, C108.2
- net GND: now also C101.1, C102.1, C103.1, C104.1, C105.1, C106.1, C107.1, C108.1
