File: XG_Mobile_USB_Hub.kicad_pcb (KiCad board)
At the start: 4 copper layers, 120 x 80 mm, 297 parts, among them J1000 USB3_A, J1100 USB_A, J1200 USB-C 24-pin 5A / 10Gbps, J1300 SWD_5, J1401 GPU_8PIN, J1402 GPU_8PIN, J1403 EPS_8PIN, J600 USB-C 24-pin 5A / 10Gbps, J700 USB-C 24-pin 5A / 10Gbps, J800 USB3_A, J900 USB3_A, Q101 CSD17577Q3A, Q102 CSD17577Q3A, Q103 CSD17577Q3A, Q104 CSD17577Q3A, Q1200 CSD17577Q3A, Q1201 CSD17577Q3A, Q201 CSD17304Q3, Q202 CSD17577Q3A, Q600 2N7002, Q700 2N7002, SW1300 Reset_Button, SW1400 SPDT 30A >=24VDC BBM, U1001 TPS259470LRPW, U101 LM51772RHAR, U1101 TPS259470LRPW, U1200 TCPP03-M20, U1201 HD3SS3212IRKSR, U1300 STM32G071KBT6N, U201 TPS40305DRCR, U301 TPS56A37RPAR, U401 TPS62130, U501 USB7206CT_KDX, U600 HD3SS3220IRNHR, U601 TPS259470LRPW, U602 74LVC1G04, U603 74LVC1G08, U700 HD3SS3220IRNHR, U701 TPS259470LRPW, U702 74LVC1G04, U703 74LVC1G08, U801 TPS259470LRPW, U901 TPS259470LRPW, Y501 25MHz CL=18pF

Commit message: eee
Parts:
- added C1304: 100nF, Capacitor_SMD:C_0603_1608Metric, B.Cu at (104.0, 122.0)
- added C1305: 1uF 6.3V, Capacitor_SMD:C_0603_1608Metric, B.Cu at (104.0, 124.0)
- added C1306: 100nF, Capacitor_SMD:C_0603_1608Metric, B.Cu at (104.0, 126.0)
- U1300: value STM32G071KBT6N -> STM32G071CBT6; footprint Package_QFP:LQFP-32_7x7mm_P0.8mm -> Package_QFP:LQFP-48_7x7mm_P0.5mm
Connections:
- U1300 pad 1: 3V3_PG -> (no net)
- U1300 pad 10: GPU1_ADC -> MCU_NRST
- U1300 pad 11: GPU2_ADC -> UP_ADC
- U1300 pad 12: EPS_ADC -> PD_IANA
- U1300 pad 13: HUB_RESET_N -> PD_RAW_ADC
- U1300 pad 14: HUB_VBUS_DET -> GPU1_ADC
- U1300 pad 15: PD_EN -> GPU2_ADC
- U1300 pad 16: PD_NRST -> EPS_ADC
- U1300 pad 17: MCU_CC2 -> HUB_RESET_N
- U1300 pad 18: MCU_CC1 -> HUB_VBUS_DET
- U1300 pad 19: GND -> PD_EN
- U1300 pad 20: TCPP_EN -> PD_NRST
- U1300 pad 21: GND -> (no net)
- U1300 pad 22: P1_ID_N -> (no net)
- U1300 pad 23: P2_ID_N -> (no net)
- U1300 pad 24: SWDIO -> (no net)
- U1300 pad 25: SWCLK -> (no net)
- U1300 pad 26: UP_FAULT_N -> (no net)
- U1300 pad 27: PD_NFLT -> MCU_CC2
- U1300 pad 28: UP_MUX_SEL -> MCU_CC1
- U1300 pad 29: UP_MUX_OEN -> GND
- U1300 pad 30: I2C_SCL -> TCPP_EN
- U1300 pad 31: I2C_SDA -> (no net)
- U1300 pad 32: CORE_PG -> GND
- U1300 pad 5: GND -> V3V3
- U1300 pad 6: MCU_NRST -> V3V3
- U1300 pad 7: UP_ADC -> GND
- U1300 pad 8: PD_IANA -> (no net)
- U1300 pad 9: PD_RAW_ADC -> (no net)
