File: XG_Mobile_USB_Hub_MCU.kicad_sch (KiCad schematic)
At the start: 39 parts, among them J1200 USB-C 24-pin 5A / 10Gbps, J1300 SWD_5, Q1200 CSD17577Q3A, Q1201 CSD17577Q3A, SW1300 Reset_Button, U1200 TCPP03-M20, U1201 HD3SS3212IRKSR, U1300 STM32G071KBT6N

Commit message: ddee
Parts:
- C1200, C1201, C1202, C1203, C1204, C1205, C1206, C1207, C1300, C1301, C1302, C1303, R1201, R1202, R1203, R1204, R1205, R1206, R1207, R1208, R1209, R1300, R1301, R1302, R1303, R1304: MPN SELECTION_REQUIRED -> (none); Part_Number (none) -> SELECTION_REQUIRED
- D1200, D1201, D1202: MPN TPD4E05U06DQAR -> (none); Part_Number (none) -> TPD4E05U06DQAR
- D1203: MPN SMBJ22CA -> (none); Part_Number (none) -> SMBJ22CA
- J1200: MPN CONNECTOR_SELECTION_REQUIRED -> (none); Part_Number (none) -> CONNECTOR_SELECTION_REQUIRED
- J1300: MPN SWD 1x5 2.54mm -> (none); Part_Number (none) -> SWD 1x5 2.54mm
- Q1200, Q1201: MPN CSD17577Q3A -> (none); Part_Number (none) -> CSD17577Q3A
- R1200: MPN WSL25127L000FEA -> (none); Part_Number (none) -> WSL25127L000FEA
- SW1300: MPN RESET_SWITCH_SELECTION_REQUIRED -> (none); Part_Number (none) -> RESET_SWITCH_SELECTION_REQUIRED
- U1200: MPN TCPP03-M20 -> (none); Part_Number (none) -> TCPP03-M20
- U1201: LCSC (none) -> C544517; MPN HD3SS3212IRKSR -> (none); Part_Number (none) -> HD3SS3212IRKSR
- U1300: LCSC (none) -> C529349; MPN STM32G071KBT6N -> (none); Part_Number (none) -> STM32G071KBT6N

Commit message: eee
Parts:
- added C1304, C1306: 100nF, Capacitor_SMD:C_0603_1608Metric, symbol Daughterboard:C
- added C1305: 1uF 6.3V, Capacitor_SMD:C_0603_1608Metric, symbol Daughterboard:C
- U1300: value STM32G071KBT6N -> STM32G071CBT6; footprint Package_QFP:LQFP-32_7x7mm_P0.8mm -> Package_QFP:LQFP-48_7x7mm_P0.5mm; symbol Daughterboard:STM32G071KBT6N -> Daughterboard:STM32G071CBT6; LCSC C529349 -> C432212; Part_Number STM32G071KBT6N -> STM32G071CBT6
Connections:
- net 3V3_PG: now also U1300.48 (PB9); no longer U1300.1 (PB9)
- net CORE_PG: now also U1300.47 (PB8); no longer U1300.32 (PB8)
- net EPS_ADC: now also U1300.16 (PA5); no longer U1300.12 (PA5)
- net GND: now also U1300.29 (PA9/UCPD1_DBCC1), U1300.32 (PA10/UCPD1_DBCC2), U1300.7 (VSS/VSSA), C1304.2, C1305.2, C1306.2; no longer U1300.19 (PA9/UCPD1_DBCC1), U1300.21 (PA10/UCPD1_DBCC2), U1300.5 (VSS)
- net GPU1_ADC: now also U1300.14 (PA3); no longer U1300.10 (PA3)
- net GPU2_ADC: now also U1300.15 (PA4); no longer U1300.11 (PA4)
- net HUB_RESET_N: now also U1300.17 (PA6); no longer U1300.13 (PA6)
- net HUB_VBUS_DET: now also U1300.18 (PA7); no longer U1300.14 (PA7)
- net I2C_SCL: now also U1300.45 (PB6); no longer U1300.30 (PB6)
- net I2C_SDA: now also U1300.46 (PB7); no longer U1300.31 (PB7)
- net MCU_CC1: now also U1300.28 (PA8); no longer U1300.18 (PA8)
- net MCU_CC2: now also U1300.27 (PB15); no longer U1300.17 (PB15)
- net MCU_NRST: now also U1300.10 (PF2-NRST); no longer U1300.6 (PF2)
- net P1_ID_N: now also U1300.33 (PA11[PA9]); no longer U1300.22 (PA9/PA11)
- net P2_ID_N: now also U1300.34 (PA12[PA10]); no longer U1300.23 (PA10/PA12)
- net PD_EN: now also U1300.19 (PB0); no longer U1300.15 (PB0)
- net PD_IANA: now also U1300.12 (PA1); no longer U1300.8 (PA1)
- net PD_NFLT: now also U1300.39 (PD1/UCPD2_DBCC1); no longer U1300.27 (PD1)
- net PD_NRST: now also U1300.20 (PB1); no longer U1300.16 (PB1)
- net PD_RAW_ADC: now also U1300.13 (PA2); no longer U1300.9 (PA2)
- net SWCLK: now also U1300.36 (PA14-BOOT0); no longer U1300.25 (PA14)
- net SWDIO: now also U1300.35 (PA13); no longer U1300.24 (PA13)
- net TCPP_EN: now also U1300.30 (PC6); no longer U1300.20 (PC6)
- net UP_ADC: now also U1300.11 (PA0); no longer U1300.7 (PA0)
- net UP_FAULT_N: now also U1300.38 (PD0); no longer U1300.26 (PD0)
- net UP_MUX_OEN: now also U1300.41 (PD3/UCPD2_DBCC2); no longer U1300.29 (PD3)
- net UP_MUX_SEL: now also U1300.40 (PD2); no longer U1300.28 (PD2)
- net V3V3: now also U1300.5 (VREF+), U1300.6 (VDD/VDDA), C1304.1, C1305.1, C1306.1
- no-connect marks 21 -> 35
Other:
- note added: "STM32G071CBT6 LQFP48: PA8(28)=UCPD1_CC1, PB15(27)=UCPD1_CC2, PB6(45)/PB7(46)=I2C1. Source-only: UCPD1 dead-battery pins 29/32 grounded. Disable BOTH UCPD dead-battery functions before GPIO use. VBAT and VREF+ tied to 3.3 V; internal VREFBUF must stay disabled. Preserve NRST and SWD; firmware required."
- note removed: "STM32G071KBT6N LQFP32: PA8=UCPD1_CC1, PB15=UCPD1_CC2, PB6/PB7=I2C1, PA13/PA14=SWD. Source-only power path. UCPD dead-battery pins grounded; disable dead-battery function in firmware. Boot from flash using option bytes; preserve NRST function. Firmware required; no PD stack is generated here."
- moved on the sheet: C1200, C1201, C1202, C1203, C1204, C1205, C1206, C1207, C1300, C1301, C1302, C1303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
