File: XG_Mobile_USB_Hub_Power.kicad_sch (KiCad schematic)
At the start: 93 parts, among them J1401 GPU_8PIN, J1402 GPU_8PIN, J1403 EPS_8PIN, Q101 CSD17577Q3A, Q102 CSD17577Q3A, Q103 CSD17577Q3A, Q104 CSD17577Q3A, Q201 CSD17304Q3, Q202 CSD17577Q3A, SW1400 SPDT 30A >=24VDC BBM, U101 LM51772RHAR, U201 TPS40305DRCR, U301 TPS56A37RPAR, U401 TPS62130

Commit message: ddee
Parts:
- C101: MPN C0805C181K5GACTU -> (none); Part_Number (none) -> C0805C181K5GACTU
- C102: MPN GRM188R71C124KA01D -> (none); Part_Number (none) -> GRM188R71C124KA01D
- C103: MPN CC0402JRNPO8BN221 -> (none); Part_Number (none) -> CC0402JRNPO8BN221
- C104: MPN GRM155R61C333KA01D -> (none); Part_Number (none) -> GRM155R61C333KA01D
- C105, C106: MPN GRM188R60J226MEA0D -> (none); Part_Number (none) -> GRM188R60J226MEA0D
- C107, C108, C304: MPN EMK107B7104KA-T -> (none); Part_Number (none) -> EMK107B7104KA-T
- C109, C1401, C1402, C1403, C1404, C402, C405, R106, R107, R108, R1400, R1401, R1402, R1403, R1404, R1405, R401, R402, R403: MPN SELECTION_REQUIRED -> (none); Part_Number (none) -> SELECTION_REQUIRED
- C110: MPN MSAST32NSB5106KTNA01 -> (none); Part_Number (none) -> MSAST32NSB5106KTNA01
- C111: MPN 25SVPF27MX -> (none); Part_Number (none) -> 25SVPF27MX
- C112, C113: MPN 35SVPF120M -> (none); Part_Number (none) -> 35SVPF120M
- C114, C115: MPN C3225X7R1H106M250AC -> (none); Part_Number (none) -> C3225X7R1H106M250AC
- C1400: MPN INPUT_BULK_CAP_SELECTION_REQUIRED -> (none); Part_Number (none) -> INPUT_BULK_CAP_SELECTION_REQUIRED
- C201, C202, C203, C401: MPN GRM31CR71E106KA12L -> (none); Part_Number (none) -> GRM31CR71E106KA12L
- C204: MPN C1005X5R1E105K050BC -> (none); Part_Number (none) -> C1005X5R1E105K050BC
- C205: MPN GRM21BR71A225KA01L -> (none); Part_Number (none) -> GRM21BR71A225KA01L
- C206: MPN GRM155R71C104KA88D -> (none); Part_Number (none) -> GRM155R71C104KA88D
- C207: MPN C3216X5R1A107M160AC -> (none); Part_Number (none) -> C3216X5R1A107M160AC
- C208: MPN GRM033R71A332KA01D -> (none); Part_Number (none) -> GRM033R71A332KA01D
- C209: MPN GRM0335C1H121JA01D -> (none); Part_Number (none) -> GRM0335C1H121JA01D
- C210: MPN C0603C432J5GAC7867 -> (none); Part_Number (none) -> C0603C432J5GAC7867
- C211: MPN GRM1555C1H102JA01J -> (none); Part_Number (none) -> GRM1555C1H102JA01J
- C301, C302: MPN MSAST21GBB5106MTNA01 -> (none); Part_Number (none) -> MSAST21GBB5106MTNA01
- C303: MPN C0603C104M3VACTU -> (none); Part_Number (none) -> C0603C104M3VACTU
- C305, C306: MPN C3225X5R1C156M250AA -> (none); Part_Number (none) -> C3225X5R1C156M250AA
- C307: MPN C0603C151K3GACTU -> (none); Part_Number (none) -> C0603C151K3GACTU
- C308: MPN GRM155R71C223KA01D -> (none); Part_Number (none) -> GRM155R71C223KA01D
- C403, C404: MPN GRM21BR60J226ME39L -> (none); Part_Number (none) -> GRM21BR60J226ME39L
- D1400: MPN SMBJ13CA -> (none); Part_Number (none) -> SMBJ13CA
- F1401, F1402, F1403: MPN FUSE_AND_HOLDER_SELECTION_REQUIRED -> (none); Part_Number (none) -> FUSE_AND_HOLDER_SELECTION_REQUIRED
- J1401, J1402: MPN PCIe_GPU_8PIN_KEYED_HEADER_SELECTION_REQUIRED -> (none); Part_Number (none) -> PCIe_GPU_8PIN_KEYED_HEADER_SELECTION_REQUIRED
- J1403: MPN EPS_CPU_8PIN_KEYED_HEADER_SELECTION_REQUIRED -> (none); Part_Number (none) -> EPS_CPU_8PIN_KEYED_HEADER_SELECTION_REQUIRED
- L101: MPN APS1040M2R2A -> (none); Part_Number (none) -> APS1040M2R2A
- L201: MPN XAL7070-801MEB -> (none); Part_Number (none) -> XAL7070-801MEB
- L301: MPN VLP8040T-2R2N -> (none); Part_Number (none) -> VLP8040T-2R2N
- L401: MPN XAL5030-222MEC -> (none); Part_Number (none) -> XAL5030-222MEC
- Q101, Q102, Q103, Q104, Q202: MPN CSD17577Q3A -> (none); Part_Number (none) -> CSD17577Q3A
- Q201: MPN CSD17304Q3 -> (none); Part_Number (none) -> CSD17304Q3
- R101: MPN WSR22L000FEA -> (none); Part_Number (none) -> WSR22L000FEA
- R102, R103: MPN CRCW060310R0FKEA -> (none); Part_Number (none) -> CRCW060310R0FKEA
- R104: MPN RC0603FR-0751KL -> (none); Part_Number (none) -> RC0603FR-0751KL
- R105: MPN CRCW04024K75FKED -> (none); Part_Number (none) -> CRCW04024K75FKED
- R201, R304: MPN CRCW0402100KFKED -> (none); Part_Number (none) -> CRCW0402100KFKED
- R202: MPN CRCW04027K50FKED -> (none); Part_Number (none) -> CRCW04027K50FKED
- R203, R302: MPN RC0201FR-0710KL -> (none); Part_Number (none) -> RC0201FR-0710KL
- R204: MPN CRCW04021K37FKED -> (none); Part_Number (none) -> CRCW04021K37FKED
- R205: MPN CRCW04022K26FKED -> (none); Part_Number (none) -> CRCW04022K26FKED
- R206: MPN CRCW0402274RFKED -> (none); Part_Number (none) -> CRCW0402274RFKED
- R301: MPN CRCW080545K3FKEA -> (none); Part_Number (none) -> CRCW080545K3FKEA
- R303: MPN CRCW040252K3FKED -> (none); Part_Number (none) -> CRCW040252K3FKED
- SW1400: MPN DC_POWER_SELECTOR_SELECTION_REQUIRED -> (none); Part_Number (none) -> DC_POWER_SELECTOR_SELECTION_REQUIRED
- U101: MPN LM51772RHAR -> (none); Part_Number (none) -> LM51772RHAR
- U201: LCSC (none) -> C140285; MPN TPS40305DRCR -> (none); Part_Number (none) -> TPS40305DRCR
- U301: LCSC (none) -> C22392669; MPN TPS56A37RPAR -> (none); Part_Number (none) -> TPS56A37RPAR
- U401: LCSC (none) -> C43590; MPN TPS62130 -> (none); Part_Number (none) -> TPS62130RGTR

Commit message: eee
Other:
- moved on the sheet: C101, C102, C103, C104, C105, C106, C107, C108, C109, C110, C111, C112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
