File: XG_Mobile_USB_Hub_USB_Hub.kicad_sch (KiCad schematic)
At the start: 165 parts, among them J1000 USB3_A, J1100 USB_A, J600 USB-C 24-pin 5A / 10Gbps, J700 USB-C 24-pin 5A / 10Gbps, J800 USB3_A, J900 USB3_A, Q600 2N7002, Q700 2N7002, U1001 TPS259470LRPW, U1101 TPS259470LRPW, U501 USB7206CT_KDX, U600 HD3SS3220IRNHR, U601 TPS259470LRPW, U602 74LVC1G04, U603 74LVC1G08, U700 HD3SS3220IRNHR, U701 TPS259470LRPW, U702 74LVC1G04, U703 74LVC1G08, U801 TPS259470LRPW, U901 TPS259470LRPW, Y501 25MHz CL=18pF

Commit message: ddee
Parts:
- C1001, C1002, C1003, C1101, C1102, C1103, C501, C502, C503, C504, C505, C506, C507, C508, C509, C510, C511, C512, C513, C514, C515, C516, C517, C518, C519, C520, C521, C522, C523, C524, C525, C526, C527, C528, C529, C530, C531, C532, C533, C534, C601, C602, C603, C604, C605, C606, C607, C608, C701, C702, C703, C704, C705, C706, C707, C708, C801, C802, C803, C901, C902, C903, R1001, R1002, R1003, R1101, R1102, R1103, R501, R502, R503, R504, R505, R506, R507, R508, R509, R510, R511, R512, R513, R514, R515, R516, R517, R518, R519, R520, R521, R522, R523, R524, R601, R602, R603, R604, R605, R606, R607, R608, R609, R610, R611, R701, R702, R703, R704, R705, R706, R707, R708, R709, R710, R711, R801, R802, R803, R901, R902, R903: MPN SELECTION_REQUIRED -> (none); Part_Number (none) -> SELECTION_REQUIRED
- C1004, C1104, C804, C904: MPN USB_A_BULK_CAP_SELECTION_REQUIRED -> (none); Part_Number (none) -> USB_A_BULK_CAP_SELECTION_REQUIRED
- D1000, D1001, D1100, D600, D601, D602, D700, D701, D702, D800, D801, D900, D901: MPN TPD4E05U06DQAR -> (none); Part_Number (none) -> TPD4E05U06DQAR
- D1009, D1109, D609, D709, D809, D909: MPN SMBJ5.0CA -> (none); Part_Number (none) -> SMBJ5.0CA
- J1000, J800, J900: MPN USB3_A_CONNECTOR_SELECTION_REQUIRED -> (none); Part_Number (none) -> USB3_A_CONNECTOR_SELECTION_REQUIRED
- J1100: MPN USB_A_CONNECTOR_SELECTION_REQUIRED -> (none); Part_Number (none) -> USB_A_CONNECTOR_SELECTION_REQUIRED
- J600, J700: MPN CONNECTOR_SELECTION_REQUIRED -> (none); Part_Number (none) -> CONNECTOR_SELECTION_REQUIRED
- Q600, Q700: MPN 2N7002 -> (none); Part_Number (none) -> 2N7002
- U1001, U1101, U601, U701, U801, U901: MPN TPS259470LRPW -> (none); Part_Number (none) -> TPS259470LRPW
- U501: MPN USB7206CT/KDX -> (none); Part_Number (none) -> USB7206CT/KDX
- U600, U700: MPN HD3SS3220IRNHR -> (none); Part_Number (none) -> HD3SS3220IRNHR
- U602, U702: MPN SN74LVC1G04DBVR -> (none); Part_Number (none) -> SN74LVC1G04DBVR
- U603, U703: MPN SN74LVC1G08DBVR -> (none); Part_Number (none) -> SN74LVC1G08DBVR
- Y501: MPN ABM8-25.000MHZ-B2-T -> (none); Part_Number (none) -> ABM8-25.000MHZ-B2-T

Commit message: eee
Other:
- moved on the sheet: C1001, C1002, C1003, C1004, C1101, C1102, C1103, C1104, C501, C601, C602, C603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
