File: USB_C_Daughterboard/Hub.kicad_sch (KiCad schematic)
At the start: 28 parts, among them U501 USB7206CT_KDX, Y501 25MHz CL=18pF

Commit message: Add USB hub PCB draft and teardrop updates
Rename the KiCad project to XG_Mobile_USB_Hub and add the unrouted PCB placement draft, generator, previews and validation reports.

Refresh schematic footprints, documentation and archive. Include the pending teardrop plugin changes, tests and reference images.
Parts:
- U501: footprint (none) -> Package_DFN_QFN:VQFN-100-1EP_12x12mm_P0.4mm_EP8x8mm
