File: USB_C_Daughterboard/Power_Core.kicad_sch (KiCad schematic)
At the start: 10 parts, among them U401 TPS62130

Commit message: Add USB hub PCB draft and teardrop updates
Rename the KiCad project to XG_Mobile_USB_Hub and add the unrouted PCB placement draft, generator, previews and validation reports.

Refresh schematic footprints, documentation and archive. Include the pending teardrop plugin changes, tests and reference images.
Parts:
- C403, C404: footprint Capacitor_SMD:C_0603_1608Metric -> Capacitor_SMD:C_0805_2012Metric
