File: USB_C_Daughterboard/USB_C1.kicad_sch (KiCad schematic)
At the start: 29 parts, among them J600 USB-C 24-pin 5A / 10Gbps, Q600 2N7002, U600 HD3SS3220IRNHR, U601 TPS259470LRPW, U602 74LVC1G04, U603 74LVC1G08

Commit message: Add USB hub PCB draft and teardrop updates
Rename the KiCad project to XG_Mobile_USB_Hub and add the unrouted PCB placement draft, generator, previews and validation reports.

Refresh schematic footprints, documentation and archive. Include the pending teardrop plugin changes, tests and reference images.
Parts:
- U600: footprint (none) -> Package_DFN_QFN:Texas_RNH0030A_WQFN-30-1EP_2.5x4.5mm_P0.4mm_EP1.2x3.2mm
