File: USB_C_Daughterboard/USB_C2.kicad_sch (KiCad schematic)
At the start: 29 parts, among them J700 USB-C 24-pin 5A / 10Gbps, Q700 2N7002, U700 HD3SS3220IRNHR, U701 TPS259470LRPW, U702 74LVC1G04, U703 74LVC1G08

Commit message: Add USB hub PCB draft and teardrop updates
Rename the KiCad project to XG_Mobile_USB_Hub and add the unrouted PCB placement draft, generator, previews and validation reports.

Refresh schematic footprints, documentation and archive. Include the pending teardrop plugin changes, tests and reference images.
Parts:
- U700: footprint (none) -> Package_DFN_QFN:Texas_RNH0030A_WQFN-30-1EP_2.5x4.5mm_P0.4mm_EP1.2x3.2mm
