File: USB_C_Daughterboard/XG_Mobile_USB_Hub.kicad_sch (KiCad schematic)
At the start: 0 parts

Commit message: Consolidate USB hub schematics into three child sheets
Group power supplies and inputs, MCU and upstream PD control, and hub/downstream ports into three child schematics.

Preserve component identities, connectivity and PCB placement while updating hierarchy links. Refresh generators, validation, BOM, ERC, documentation, PDF/SVG exports and archive.
Other:
- removed sheet 1.15 V / 3 A - USB7206C core
- removed sheet 12 V input - two GPU 8-pin OR one EPS 8-pin
- removed sheet 3.3 V / 4 A - TPS56A37
- removed sheet 5 V / 12 A - TPS40305
- removed sheet Downstream Type-A 1 - SuperSpeed / 900 mA
- removed sheet Downstream Type-A 2 - SuperSpeed / 900 mA
- removed sheet Downstream Type-A 3 - SuperSpeed / 900 mA
- removed sheet Downstream Type-A 4 - USB 2.0 / 500 mA
- removed sheet Downstream Type-C 1 - 5 V / 3 A
- removed sheet Downstream Type-C 2 - 5 V / 3 A
- removed sheet Hub decoupling and transmit coupling
- removed sheet LM51772 - programmable 5-20 V / 100 W
- removed sheet STM32G071 - USB-PD policy and power control
- removed sheet USB7206C - six downstream ports
- removed sheet Upstream Type-C - USB data UFP / PD source
- added sheet MCU and Upstream PD Control (MCU.kicad_sch)
- added sheet Power Supplies and Inputs (Power.kicad_sch)
- added sheet USB Hub and Downstream Ports (USB_Hub.kicad_sch)
- title: USB C Daughterboard -> XG Mobile USB Hub
Changed lines of the file:
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@@
 (kicad_sch (version 20231120) (generator "eeschema")
- (paper "A2")
-      (title_block (title "USB C Daughterboard") (rev "DRAFT A")
+ (paper "A3")
+      (title_block (title "XG Mobile USB Hub") (rev "DRAFT A")
         (comment 1 "Engineering draft - not released for manufacture")
         (comment 2 "12 V input / 100 W upstream USB-PD / 2 USB-C + 4 USB-A downstream"))
-(sheet (at 20 55) (size 160 30) (stroke (width 0) (type default)) (fill (color 0 0 0 0))
-          (property "Sheetname" "3.3 V / 4 A - TPS56A37" (at 20 53.73 0) (effects (font (size 1.27 1.27)) (justify left bottom)))
-          (property "Sheetfile" "Power_3V3.kicad_sch" (at 20 86.27 0) (effects (font (size 1.27 1.27)) (justify left top)))
+(sheet (at 20 65) (size 160 30) (stroke (width 0) (type default)) (fill (color 0 0 0 0))
+          (property "Sheetname" "Power Supplies and Inputs" (at 20 63.73 0) (effects (font (size 1.27 1.27)) (justify left bottom)))
+          (property "Sheetfile" "Power.kicad_sch" (at 20 96.27 0) (effects (font (size 1.27 1.27)) (justify left top)))
           (instances (project "XG_Mobile_USB_Hub" (path "/af461753-d65f-5f37-931d-eaa9a181614a" (page "2")))))
-(sheet (at 200 55) (size 160 30) (stroke (width 0) (type default)) (fill (color 0 0 0 0))
-          (property "Sheetname" "5 V / 12 A - TPS40305" (at 200 53.73 0) (effects (font (size 1.27 1.27)) (justify left bottom)))
-          (property "Sheetfile" "Power_5V.kicad_sch" (at 200 86.27 0) (effects (font (size 1.27 1.27)) (justify left top)))
+(sheet (at 20 120) (size 160 30) (stroke (width 0) (type default)) (fill (color 0 0 0 0))
+          (property "Sheetname" "MCU and Upstream PD Control" (at 20 118.73 0) (effects (font (size 1.27 1.27)) (justify left bottom)))
+          (property "Sheetfile" "MCU.kicad_sch" (at 20 151.27 0) (effects (font (size 1.27 1.27)) (justify left top)))
           (instances (project "XG_Mobile_USB_Hub" (path "/af461753-d65f-5f37-931d-eaa9a181614a" (page "3")))))
-(sheet (at 380 55) (size 160 30) (stroke (width 0) (type default)) (fill (color 0 0 0 0))
-          (property "Sheetname" "1.15 V / 3 A - USB7206C core" (at 380 53.73 0) (effects (font (size 1.27 1.27)) (justify left bottom)))
-          (property "Sheetfile" "Power_Core.kicad_sch" (at 380 86.27 0) (effects (font (size 1.27 1.27)) (justify left top)))
+(sheet (at 20 175) (size 160 30) (stroke (width 0) (type default)) (fill (color 0 0 0 0))
+          (property "Sheetname" "USB Hub and Downstream Ports" (at 20 173.73 0) (effects (font (size 1.27 1.27)) (justify left bottom)))
+          (property "Sheetfile" "USB_Hub.kicad_sch" (at 20 206.27 0) (effects (font (size 1.27 1.27)) (justify left top)))
           (instances (project "XG_Mobile_USB_Hub" (path "/af461753-d65f-5f37-931d-eaa9a181614a" (page "4")))))
-(sheet (at 20 103) (size 160 30) (stroke (width 0) (type default)) (fill (color 0 0 0 0))
-          (property "Sheetname" "USB7206C - six downstream ports" (at 20 101.73 0) (effects (font (size 1.27 1.27)) (justify left bottom)))
-          (property "Sheetfile" "Hub.kicad_sch" (at 20 134.27 0) (effects (font (size 1.27 1.27)) (justify left top)))
-          (instances (project "XG_Mobile_USB_Hub" (path "/af461753-d65f-5f37-931d-eaa9a181614a" (page "5")))))
-(sheet (at 200 103) (size 160 30) (stroke (width 0) (type default)) (fill (color 0 0 0 0))
-          (property "Sheetname" "Hub decoupling and transmit coupling" (at 200 101.73 0) (effects (font (size 1.27 1.27)) (justify left bottom)))
-          (property "Sheetfile" "Hub_Decoupling.kicad_sch" (at 200 134.27 0) (effects (font (size 1.27 1.27)) (justify left top)))
-          (instances (project "XG_Mobile_USB_Hub" (path "/af461753-d65f-5f37-931d-eaa9a181614a" (page "6")))))
-(sheet (at 380 103) (size 160 30) (stroke (width 0) (type default)) (fill (color 0 0 0 0))
-          (property "Sheetname" "Downstream Type-C 1 - 5 V / 3 A" (at 380 101.73 0) (effects (font (size 1.27 1.27)) (justify left bottom)))
-          (property "Sheetfile" "USB_C1.kicad_sch" (at 380 134.27 0) (effects (font (size 1.27 1.27)) (justify left top)))
-          (instances (project "XG_Mobile_USB_Hub" (path "/af461753-d65f-5f37-931d-eaa9a181614a" (page "7")))))
-(sheet (at 20 151) (size 160 30) (stroke (width 0) (type default)) (fill (color 0 0 0 0))
-          (property "Sheetname" "Downstream Type-C 2 - 5 V / 3 A" (at 20 149.73 0) (effects (font (size 1.27 1.27)) (justify left bottom)))
-          (property "Sheetfile" "USB_C2.kicad_sch" (at 20 182.27 0) (effects (font (size 1.27 1.27)) (justify left top)))
-          (instances (project "XG_Mobile_USB_Hub" (path "/af461753-d65f-5f37-931d-eaa9a181614a" (page "8")))))
-(sheet (at 200 151) (size 160 30) (stroke (width 0) (type default)) (fill (color 0 0 0 0))
-          (property "Sheetname" "Downstream Type-A 1 - SuperSpeed / 900 mA" (at 200 149.73 0) (effects (font (size 1.27 1.27)) (justify left bottom)))
-          (property "Sheetfile" "USB_A1.kicad_sch" (at 200 182.27 0) (effects (font (size 1.27 1.27)) (justify left top)))
-          (instances (project "XG_Mobile_USB_Hub" (path "/af461753-d65f-5f37-931d-eaa9a181614a" (page "9")))))
-(sheet (at 380 151) (size 160 30) (stroke (width 0) (type default)) (fill (color 0 0 0 0))
-          (property "Sheetname" "Downstream Type-A 2 - SuperSpeed / 900 mA" (at 380 149.73 0) (effects (font (size 1.27 1.27)) (justify left bottom)))
-          (property "Sheetfile" "USB_A2.kicad_sch" (at 380 182.27 0) (effects (font (size 1.27 1.27)) (justify left top)))
-          (instances (project "XG_Mobile_USB_Hub" (path "/af461753-d65f-5f37-931d-eaa9a181614a" (page "10")))))
-(sheet (at 20 199) (size 160 30) (stroke (width 0) (type default)) (fill (color 0 0 0 0))
-          (property "Sheetname" "Downstream Type-A 3 - SuperSpeed / 900 mA" (at 20 197.73 0) (effects (font (size 1.27 1.27)) (justify left bottom)))
-          (property "Sheetfile" "USB_A3.kicad_sch" (at 20 230.27 0) (effects (font (size 1.27 1.27)) (justify left top)))
-          (instances (project "XG_Mobile_USB_Hub" (path "/af461753-d65f-5f37-931d-eaa9a181614a" (page "11")))))
-(sheet (at 200 199) (size 160 30) (stroke (width 0) (type default)) (fill (color 0 0 0 0))
-          (property "Sheetname" "Downstream Type-A 4 - USB 2.0 / 500 mA" (at 200 197.73 0) (effects (font (size 1.27 1.27)) (justify left bottom)))
-          (property "Sheetfile" "USB_A4.kicad_sch" (at 200 230.27 0) (effects (font (size 1.27 1.27)) (justify left top)))
-          (instances (project "XG_Mobile_USB_Hub" (path "/af461753-d65f-5f37-931d-eaa9a181614a" (page "12")))))
-(sheet (at 380 199) (size 160 30) (stroke (width 0) (type default)) (fill (color 0 0 0 0))
-          (property "Sheetname" "LM51772 - programmable 5-20 V / 100 W" (at 380 197.73 0) (effects (font (size 1.27 1.27)) (justify left bottom)))
-          (property "Sheetfile" "PD_BuckBoost.kicad_sch" (at 380 230.27 0) (effects (font (size 1.27 1.27)) (justify left top)))
-          (instances (project "XG_Mobile_USB_Hub" (path "/af461753-d65f-5f37-931d-eaa9a181614a" (page "13")))))
-(sheet (at 20 247) (size 160 30) (stroke (width 0) (type default)) (fill (color 0 0 0 0))
-          (property "Sheetname" "Upstream Type-C - USB data UFP / PD source" (at 20 245.73 0) (effects (font (size 1.27 1.27)) (justify left bottom)))
-          (property "Sheetfile" "USB_Upstream.kicad_sch" (at 20 278.27 0) (effects (font (size 1.27 1.27)) (justify left top)))
-          (instances (project "XG_Mobile_USB_Hub" (path "/af461753-d65f-5f37-931d-eaa9a181614a" (page "14")))))
-(sheet (at 200 247) (size 160 30) (stroke (width 0) (type default)) (fill (color 0 0 0 0))
-          (property "Sheetname" "STM32G071 - USB-PD policy and power control" (at 200 245.73 0) (effects (font (size 1.27 1.27)) (justify left bottom)))
-          (property "Sheetfile" "PD_MCU.kicad_sch" (at 200 278.27 0) (effects (font (size 1.27 1.27)) (justify left top)))
-          (instances (project "XG_Mobile_USB_Hub" (path "/af461753-d65f-5f37-931d-eaa9a181614a" (page "15")))))
-(sheet (at 380 247) (size 160 30) (stroke (width 0) (type default)) (fill (color 0 0 0 0))
-          (property "Sheetname" "12 V input - two GPU 8-pin OR one EPS 8-pin" (at 380 245.73 0) (effects (font (size 1.27 1.27)) (justify left bottom)))
-          (property "Sheetfile" "Power_Input.kicad_sch" (at 380 278.27 0) (effects (font (size 1.27 1.27)) (justify left top)))
-          (instances (project "XG_Mobile_USB_Hub" (path "/af461753-d65f-5f37-931d-eaa9a181614a" (page "16")))))
 (text "USB-C DAUGHTERBOARD / ENGINEERING DRAFT" (at 20 15 0) (effects (font (size 3 3)) (justify left top)))
 (text "Upstream: USB-C, USB 3.2 Gen 2 data UFP, USB-PD power source, 20 V / 5 A maximum.\nDownstream: 2 Type-C + 3 Type-A SuperSpeed, 1 Type-A USB 2.0.\nUse two GPU power inputs OR one EPS input. Not for simultaneous independent supplies." (at 20 24 0) (effects (font (size 1.27 1.27)) (justify left top)))
